File: osab.sch (KiCad schematic (older format))
At the start: 88 parts, among them CON1 TF-01A, CON2 PJ-3420-A-SMT, CON3 TYPE-C-31-M-12, Q1 BC847B, SW1 PPP, SW10 RESET, SW2 VOL-, SW3 VOL+, SW4 CHAP-, SW5 CHAP+, SW6 OT/NT, SW7 BOOK-, SW8 BOOK+, SW9 BUTTON_LOCK, U1 VS1000, U2 ME6211C33M5G-N, U3 25LC640A, U4 TP4055, U5 MF5853CS, U6 TCS7191, Y1 12MHz

Commit message: production: 100n caps replaced with 0603 Samsung
Parts:
- C10, C12, C14, C15, C16, C6, C8: Link https://lcsc.com/product-detail/Multilayer-Ceramic-Capacitors-MLCC-SMD-SMT_CCTC-TCC0805X7R104K500DT_C282732.html -> https://lcsc.com/product-detail/Multilayer-Ceramic-Capacitors-MLCC-SMD-SMT_Samsung-Electro-Mechanics-CL10B104KB8NNNC_C1591.html; MPN TCC0805X7R104K500DT -> CL10B104KB8NNNC
Changed lines of the file:
@@
 F 1 "100n X7R" H 6250 2650 50  0000 L CNN
 F 2 "Capacitor_SMD:C_0603_1608Metric" H 6488 2600 50  0001 C CNN
-F 3 "https://datasheet.lcsc.com/szlcsc/1810261827_CCTC-TCC0805X7R104K500DT_C282732.pdf" H 6450 2750 50  0001 C CNN
+F 3 "https://datasheet.lcsc.com/lcsc/1811021431_Samsung-Electro-Mechanics-CL10B104KB8NNNC_C1591.pdf" H 6450 2750 50  0001 C CNN
 F 4 "Included in KiCad" H 6450 2750 50  0001 C CNN "3D-model"
-F 5 "https://lcsc.com/product-detail/Multilayer-Ceramic-Capacitors-MLCC-SMD-SMT_CCTC-TCC0805X7R104K500DT_C282732.html" H 6450 2750 50  0001 C CNN "Link"
-F 6 "TCC0805X7R104K500DT" H 6450 2750 50  0001 C CNN "MPN"
+F 5 "https://lcsc.com/product-detail/Multilayer-Ceramic-Capacitors-MLCC-SMD-SMT_Samsung-Electro-Mechanics-CL10B104KB8NNNC_C1591.html" H 6450 2750 50  0001 C CNN "Link"
+F 6 "CL10B104KB8NNNC" H 6450 2750 50  0001 C CNN "MPN"
 	1    6450 2750
 	1    0    0    -1
@@
 F 1 "100n X7R" H 6000 2950 50  0000 L CNN
 F 2 "Capacitor_SMD:C_0603_1608Metric" H 6238 2600 50  0001 C CNN
-F 3 "https://datasheet.lcsc.com/szlcsc/1810261827_CCTC-TCC0805X7R104K500DT_C282732.pdf" H 6200 2750 50  0001 C CNN
+F 3 "https://datasheet.lcsc.com/lcsc/1811021431_Samsung-Electro-Mechanics-CL10B104KB8NNNC_C1591.pdf" H 6200 2750 50  0001 C CNN
 F 4 "Included in KiCad" H 6200 2750 50  0001 C CNN "3D-model"
-F 5 "https://lcsc.com/product-detail/Multilayer-Ceramic-Capacitors-MLCC-SMD-SMT_CCTC-TCC0805X7R104K500DT_C282732.html" H 6200 2750 50  0001 C CNN "Link"
-F 6 "TCC0805X7R104K500DT" H 6200 2750 50  0001 C CNN "MPN"
+F 5 "https://lcsc.com/product-detail/Multilayer-Ceramic-Capacitors-MLCC-SMD-SMT_Samsung-Electro-Mechanics-CL10B104KB8NNNC_C1591.html" H 6200 2750 50  0001 C CNN "Link"
+F 6 "CL10B104KB8NNNC" H 6200 2750 50  0001 C CNN "MPN"
 	1    6200 2750
 	1    0    0    -1
@@
 F 1 "100n X7R" H 4950 5400 50  0000 L CNN
 F 2 "Capacitor_SMD:C_0603_1608Metric" H 5188 5350 50  0001 C CNN
-F 3 "https://datasheet.lcsc.com/szlcsc/1810261827_CCTC-TCC0805X7R104K500DT_C282732.pdf" H 5150 5500 50  0001 C CNN
+F 3 "https://datasheet.lcsc.com/lcsc/1811021431_Samsung-Electro-Mechanics-CL10B104KB8NNNC_C1591.pdf" H 5150 5500 50  0001 C CNN
 F 4 "Included in KiCad" H 5150 5500 50  0001 C CNN "3D-model"
-F 5 "https://lcsc.com/product-detail/Multilayer-Ceramic-Capacitors-MLCC-SMD-SMT_CCTC-TCC0805X7R104K500DT_C282732.html" H 5150 5500 50  0001 C CNN "Link"
-F 6 "TCC0805X7R104K500DT" H 5150 5500 50  0001 C CNN "MPN"
+F 5 "https://lcsc.com/product-detail/Multilayer-Ceramic-Capacitors-MLCC-SMD-SMT_Samsung-Electro-Mechanics-CL10B104KB8NNNC_C1591.html" H 5150 5500 50  0001 C CNN "Link"
+F 6 "CL10B104KB8NNNC" H 5150 5500 50  0001 C CNN "MPN"
 	1    5150 5500
 	1    0    0    -1
@@
 F 1 "100n X7R" H 5450 5400 50  0000 L CNN
 F 2 "Capacitor_SMD:C_0603_1608Metric" H 5438 5350 50  0001 C CNN
-F 3 "https://datasheet.lcsc.com/szlcsc/1810261827_CCTC-TCC0805X7R104K500DT_C282732.pdf" H 5400 5500 50  0001 C CNN
+F 3 "https://datasheet.lcsc.com/lcsc/1811021431_Samsung-Electro-Mechanics-CL10B104KB8NNNC_C1591.pdf" H 5400 5500 50  0001 C CNN
 F 4 "Included in KiCad" H 5400 5500 50  0001 C CNN "3D-model"
-F 5 "https://lcsc.com/product-detail/Multilayer-Ceramic-Capacitors-MLCC-SMD-SMT_CCTC-TCC0805X7R104K500DT_C282732.html" H 5400 5500 50  0001 C CNN "Link"
-F 6 "TCC0805X7R104K500DT" H 5400 5500 50  0001 C CNN "MPN"
+F 5 "https://lcsc.com/product-detail/Multilayer-Ceramic-Capacitors-MLCC-SMD-SMT_Samsung-Electro-Mechanics-CL10B104KB8NNNC_C1591.html" H 5400 5500 50  0001 C CNN "Link"
+F 6 "CL10B104KB8NNNC" H 5400 5500 50  0001 C CNN "MPN"
 	1    5400 5500
 	1    0    0    -1
@@
 F 1 "100n X7R" H 5450 5000 50  0000 L CNN
 F 2 "Capacitor_SMD:C_0603_1608Metric" H 5688 5000 50  0001 C CNN
-F 3 "https://datasheet.lcsc.com/szlcsc/1810261827_CCTC-TCC0805X7R104K500DT_C282732.pdf" H 5650 5150 50  0001 C CNN
+F 3 "https://datasheet.lcsc.com/lcsc/1811021431_Samsung-Electro-Mechanics-CL10B104KB8NNNC_C1591.pdf" H 5650 5150 50  0001 C CNN
 F 4 "Included in KiCad" H 5650 5150 50  0001 C CNN "3D-model"
-F 5 "https://lcsc.com/product-detail/Multilayer-Ceramic-Capacitors-MLCC-SMD-SMT_CCTC-TCC0805X7R104K500DT_C282732.html" H 5650 5150 50  0001 C CNN "Link"
-F 6 "TCC0805X7R104K500DT" H 5650 5150 50  0001 C CNN "MPN"
+F 5 "https://lcsc.com/product-detail/Multilayer-Ceramic-Capacitors-MLCC-SMD-SMT_Samsung-Electro-Mechanics-CL10B104KB8NNNC_C1591.html" H 5650 5150 50  0001 C CNN "Link"
+F 6 "CL10B104KB8NNNC" H 5650 5150 50  0001 C CNN "MPN"
 	1    5650 5150
 	1    0    0    -1
@@
 F 1 "100n X7R" H 5700 5050 50  0000 L CNN
 F 2 "Capacitor_SMD:C_0603_1608Metric" H 5938 5000 50  0001 C CNN
-F 3 "https://datasheet.lcsc.com/szlcsc/1810261827_CCTC-TCC0805X7R104K500DT_C282732.pdf" H 5900 5150 50  0001 C CNN
+F 3 "https://datasheet.lcsc.com/lcsc/1811021431_Samsung-Electro-Mechanics-CL10B104KB8NNNC_C1591.pdf" H 5900 5150 50  0001 C CNN
 F 4 "Included in KiCad" H 5900 5150 50  0001 C CNN "3D-model"
-F 5 "https://lcsc.com/product-detail/Multilayer-Ceramic-Capacitors-MLCC-SMD-SMT_CCTC-TCC0805X7R104K500DT_C282732.html" H 5900 5150 50  0001 C CNN "Link"
-F 6 "TCC0805X7R104K500DT" H 5900 5150 50  0001 C CNN "MPN"
+F 5 "https://lcsc.com/product-detail/Multilayer-Ceramic-Capacitors-MLCC-SMD-SMT_Samsung-Electro-Mechanics-CL10B104KB8NNNC_C1591.html" H 5900 5150 50  0001 C CNN "Link"
+F 6 "CL10B104KB8NNNC" H 5900 5150 50  0001 C CNN "MPN"
 	1    5900 5150
 	1    0    0    -1
@@
 F 1 "100n X7R" H 5950 5000 50  0000 L CNN
 F 2 "Capacitor_SMD:C_0603_1608Metric" H 6188 5000 50  0001 C CNN
-F 3 "https://datasheet.lcsc.com/szlcsc/1810261827_CCTC-TCC0805X7R104K500DT_C282732.pdf" H 6150 5150 50  0001 C CNN
+F 3 "https://datasheet.lcsc.com/lcsc/1811021431_Samsung-Electro-Mechanics-CL10B104KB8NNNC_C1591.pdf" H 6150 5150 50  0001 C CNN
 F 4 "Included in KiCad" H 6150 5150 50  0001 C CNN "3D-model"
-F 5 "https://lcsc.com/product-detail/Multilayer-Ceramic-Capacitors-MLCC-SMD-SMT_CCTC-TCC0805X7R104K500DT_C282732.html" H 6150 5150 50  0001 C CNN "Link"
-F 6 "TCC0805X7R104K500DT" H 6150 5150 50  0001 C CNN "MPN"
+F 5 "https://lcsc.com/product-detail/Multilayer-Ceramic-Capacitors-MLCC-SMD-SMT_Samsung-Electro-Mechanics-CL10B104KB8NNNC_C1591.html" H 6150 5150 50  0001 C CNN "Link"
+F 6 "CL10B104KB8NNNC" H 6150 5150 50  0001 C CNN "MPN"
 	1    6150 5150
 	1    0    0    -1

Commit message: production: Changed MPNs for earlier cap changes
Parts:
- C1, C2: MPN CL21C220JBANNNC -> CL10C220JB8NNNC
- C11, C18, C3: MPN TCC0805X7R106K100FT -> CL10A106KP8NNNC
- C13, C17, C23, C4, C5, C7, C9: MPN 0805B105K100CT -> CL10A105KP8NNNC
Changed lines of the file:
@@
 F 4 "Included in KiCad" H 5950 2750 50  0001 C CNN "3D-model"
 F 5 "https://lcsc.com/product-detail/Multilayer-Ceramic-Capacitors-MLCC-SMD-SMT_Samsung-Electro-Mechanics-CL10A105KP8NNNC_C26413.html" H 5950 2750 50  0001 C CNN "Link"
-F 6 "0805B105K100CT" H 5950 2750 50  0001 C CNN "MPN"
+F 6 "CL10A105KP8NNNC" H 5950 2750 50  0001 C CNN "MPN"
 	1    5950 2750
 	1    0    0    -1
@@
 F 4 "Included in KiCad" H 5700 2750 50  0001 C CNN "3D-model"
 F 5 "https://lcsc.com/product-detail/Multilayer-Ceramic-Capacitors-MLCC-SMD-SMT_Samsung-Electro-Mechanics-CL10A106KP8NNNC_C19702.html" H 5700 2750 50  0001 C CNN "Link"
-F 6 "TCC0805X7R106K100FT" H 5700 2750 50  0001 C CNN "MPN"
+F 6 "CL10A106KP8NNNC" H 5700 2750 50  0001 C CNN "MPN"
 	1    5700 2750
 	1    0    0    -1
@@
 F 4 "Included in KiCad" H 5450 2750 50  0001 C CNN "3D-model"
 F 5 "https://lcsc.com/product-detail/Multilayer-Ceramic-Capacitors-MLCC-SMD-SMT_Samsung-Electro-Mechanics-CL10A105KP8NNNC_C26413.html" H 5450 2750 50  0001 C CNN "Link"
-F 6 "0805B105K100CT" H 5450 2750 50  0001 C CNN "MPN"
+F 6 "CL10A105KP8NNNC" H 5450 2750 50  0001 C CNN "MPN"
 	1    5450 2750
 	1    0    0    -1
@@
 F 4 "Included in KiCad" H 3400 1750 50  0001 C CNN "3D-model"
 F 5 "https://lcsc.com/product-detail/Multilayer-Ceramic-Capacitors-MLCC-SMD-SMT_Samsung-Electro-Mechanics-CL10A106KP8NNNC_C19702.html" H 3400 1750 50  0001 C CNN "Link"
-F 6 "TCC0805X7R106K100FT" H 3400 1750 50  0001 C CNN "MPN"
+F 6 "CL10A106KP8NNNC" H 3400 1750 50  0001 C CNN "MPN"
 	1    3400 1750
 	1    0    0    -1
@@
 F 4 "Included in KiCad" H 1250 6050 50  0001 C CNN "3D-model"
 F 5 "https://lcsc.com/product-detail/Multilayer-Ceramic-Capacitors-MLCC-SMD-SMT_Samsung-Electro-Mechanics-CL10A105KP8NNNC_C26413.html" H 1250 6050 50  0001 C CNN "Link"
-F 6 "0805B105K100CT" H 1250 6050 50  0001 C CNN "MPN"
+F 6 "CL10A105KP8NNNC" H 1250 6050 50  0001 C CNN "MPN"
 	1    1250 6050
 	1    0    0    -1
@@
 F 4 "Included in KiCad" H 2600 6050 50  0001 C CNN "3D-model"
 F 5 "https://lcsc.com/product-detail/Multilayer-Ceramic-Capacitors-MLCC-SMD-SMT_Samsung-Electro-Mechanics-CL10A105KP8NNNC_C26413.html" H 2600 6050 50  0001 C CNN "Link"
-F 6 "0805B105K100CT" H 2600 6050 50  0001 C CNN "MPN"
+F 6 "CL10A105KP8NNNC" H 2600 6050 50  0001 C CNN "MPN"
 	1    2600 6050
 	1    0    0    -1
@@
 F 4 "Included in KiCad" H 10200 4850 50  0001 C CNN "3D-model"
 F 5 "https://lcsc.com/product-detail/Multilayer-Ceramic-Capacitors-MLCC-SMD-SMT_Samsung-Electro-Mechanics-CL10A106KP8NNNC_C19702.html" H 10200 4850 50  0001 C CNN "Link"
-F 6 "TCC0805X7R106K100FT" H 10200 4850 50  0001 C CNN "MPN"
+F 6 "CL10A106KP8NNNC" H 10200 4850 50  0001 C CNN "MPN"
 	1    10200 4850
 	1    0    0    -1
@@
 F 4 "Included in KiCad" H 10400 2900 50  0001 C CNN "3D-model"
 F 5 "https://lcsc.com/product-detail/Multilayer-Ceramic-Capacitors-MLCC-SMD-SMT_Samsung-Electro-Mechanics-CL10A105KP8NNNC_C26413.html" H 10400 2900 50  0001 C CNN "Link"
-F 6 "0805B105K100CT" H 10400 2900 50  0001 C CNN "MPN"
+F 6 "CL10A105KP8NNNC" H 10400 2900 50  0001 C CNN "MPN"
 	1    10400 2900
 	0    -1   -1   0
@@
 F 4 "Included in KiCad" H 5350 3400 50  0001 C CNN "3D-model"
 F 5 "https://lcsc.com/product-detail/Multilayer-Ceramic-Capacitors-MLCC-SMD-SMT_Samsung-Electro-Mechanics-CL10A105KP8NNNC_C26413.html" H 5350 3400 50  0001 C CNN "Link"
-F 6 "0805B105K100CT" H 5350 3400 50  0001 C CNN "MPN"
+F 6 "CL10A105KP8NNNC" H 5350 3400 50  0001 C CNN "MPN"
 	1    5350 3400
 	0    1    1    0
@@
 F 4 "Included in KiCad" H 8100 4850 50  0001 C CNN "3D-model"
 F 5 "https://lcsc.com/product-detail/Multilayer-Ceramic-Capacitors-MLCC-SMD-SMT_Samsung-Electro-Mechanics-CL10A105KP8NNNC_C26413.html" H 8100 4850 50  0001 C CNN "Link"
-F 6 "0805B105K100CT" H 8100 4850 50  0001 C CNN "MPN"
+F 6 "CL10A105KP8NNNC" H 8100 4850 50  0001 C CNN "MPN"
 	1    8100 4850
 	1    0    0    -1
@@
 F 4 "Included in KiCad" H 2500 1100 50  0001 C CNN "3D-model"
 F 5 "https://lcsc.com/product-detail/Multilayer-Ceramic-Capacitors-MLCC-SMD-SMT_Samsung-Electro-Mechanics-CL10C220JB8NNNC_C1653.html" H 2500 1100 50  0001 C CNN "Link"
-F 6 "CL21C220JBANNNC" H 2500 1100 50  0001 C CNN "MPN"
+F 6 "CL10C220JB8NNNC" H 2500 1100 50  0001 C CNN "MPN"
 	1    2500 1100
 	1    0    0    -1
@@
 F 4 "Included in KiCad" H 3000 1100 50  0001 C CNN "3D-model"
 F 5 "https://lcsc.com/product-detail/Multilayer-Ceramic-Capacitors-MLCC-SMD-SMT_Samsung-Electro-Mechanics-CL10C220JB8NNNC_C1653.html" H 3000 1100 50  0001 C CNN "Link"
-F 6 "CL21C220JBANNNC" H 3000 1100 50  0001 C CNN "MPN"
+F 6 "CL10C220JB8NNNC" H 3000 1100 50  0001 C CNN "MPN"
 	1    3000 1100
 	1    0    0    -1

Commit message: production: Changed 1u from 10V to 50V
Parts:
- C13, C17, C23, C4, C5, C7, C9: Link https://lcsc.com/product-detail/Multilayer-Ceramic-Capacitors-MLCC-SMD-SMT_Samsung-Electro-Mechanics-CL10A105KP8NNNC_C26413.html -> https://lcsc.com/product-detail/Multilayer-Ceramic-Capacitors-MLCC-SMD-SMT_Samsung-Electro-Mechanics-CL10A105KB8NNNC_C15849.html; MPN CL10A105KP8NNNC -> CL10A105KB8NNNC
Changed lines of the file:
@@
 F 1 "1u X5R" H 5850 2650 50  0000 L CNN
 F 2 "Capacitor_SMD:C_0603_1608Metric" H 5988 2600 50  0001 C CNN
-F 3 "https://datasheet.lcsc.com/lcsc/1811021622_Samsung-Electro-Mechanics-CL10A105KP8NNNC_C26413.pdf" H 5950 2750 50  0001 C CNN
+F 3 "https://lcsc.com/product-detail/Multilayer-Ceramic-Capacitors-MLCC-SMD-SMT_Samsung-Electro-Mechanics-CL10A105KB8NNNC_C15849.html" H 5950 2750 50  0001 C CNN
 F 4 "Included in KiCad" H 5950 2750 50  0001 C CNN "3D-model"
-F 5 "https://lcsc.com/product-detail/Multilayer-Ceramic-Capacitors-MLCC-SMD-SMT_Samsung-Electro-Mechanics-CL10A105KP8NNNC_C26413.html" H 5950 2750 50  0001 C CNN "Link"
-F 6 "CL10A105KP8NNNC" H 5950 2750 50  0001 C CNN "MPN"
+F 5 "https://lcsc.com/product-detail/Multilayer-Ceramic-Capacitors-MLCC-SMD-SMT_Samsung-Electro-Mechanics-CL10A105KB8NNNC_C15849.html" H 5950 2750 50  0001 C CNN "Link"
+F 6 "CL10A105KB8NNNC" H 5950 2750 50  0001 C CNN "MPN"
 	1    5950 2750
 	1    0    0    -1
@@
 F 1 "1u X5R" H 5350 2650 50  0000 L CNN
 F 2 "Capacitor_SMD:C_0603_1608Metric" H 5488 2600 50  0001 C CNN
-F 3 "https://datasheet.lcsc.com/lcsc/1811021622_Samsung-Electro-Mechanics-CL10A105KP8NNNC_C26413.pdf" H 5450 2750 50  0001 C CNN
+F 3 "https://lcsc.com/product-detail/Multilayer-Ceramic-Capacitors-MLCC-SMD-SMT_Samsung-Electro-Mechanics-CL10A105KB8NNNC_C15849.html" H 5450 2750 50  0001 C CNN
 F 4 "Included in KiCad" H 5450 2750 50  0001 C CNN "3D-model"
-F 5 "https://lcsc.com/product-detail/Multilayer-Ceramic-Capacitors-MLCC-SMD-SMT_Samsung-Electro-Mechanics-CL10A105KP8NNNC_C26413.html" H 5450 2750 50  0001 C CNN "Link"
-F 6 "CL10A105KP8NNNC" H 5450 2750 50  0001 C CNN "MPN"
+F 5 "https://lcsc.com/product-detail/Multilayer-Ceramic-Capacitors-MLCC-SMD-SMT_Samsung-Electro-Mechanics-CL10A105KB8NNNC_C15849.html" H 5450 2750 50  0001 C CNN "Link"
+F 6 "CL10A105KB8NNNC" H 5450 2750 50  0001 C CNN "MPN"
 	1    5450 2750
 	1    0    0    -1
@@
 F 1 "1u X5R" H 1150 5950 50  0000 L CNN
 F 2 "Capacitor_SMD:C_0603_1608Metric" H 1288 5900 50  0001 C CNN
-F 3 "https://datasheet.lcsc.com/lcsc/1811021622_Samsung-Electro-Mechanics-CL10A105KP8NNNC_C26413.pdf" H 1250 6050 50  0001 C CNN
+F 3 "https://lcsc.com/product-detail/Multilayer-Ceramic-Capacitors-MLCC-SMD-SMT_Samsung-Electro-Mechanics-CL10A105KB8NNNC_C15849.html" H 1250 6050 50  0001 C CNN
 F 4 "Included in KiCad" H 1250 6050 50  0001 C CNN "3D-model"
-F 5 "https://lcsc.com/product-detail/Multilayer-Ceramic-Capacitors-MLCC-SMD-SMT_Samsung-Electro-Mechanics-CL10A105KP8NNNC_C26413.html" H 1250 6050 50  0001 C CNN "Link"
-F 6 "CL10A105KP8NNNC" H 1250 6050 50  0001 C CNN "MPN"
+F 5 "https://lcsc.com/product-detail/Multilayer-Ceramic-Capacitors-MLCC-SMD-SMT_Samsung-Electro-Mechanics-CL10A105KB8NNNC_C15849.html" H 1250 6050 50  0001 C CNN "Link"
+F 6 "CL10A105KB8NNNC" H 1250 6050 50  0001 C CNN "MPN"
 	1    1250 6050
 	1    0    0    -1
@@
 F 1 "1u X5R" H 2500 5950 50  0000 L CNN
 F 2 "Capacitor_SMD:C_0603_1608Metric" H 2638 5900 50  0001 C CNN
-F 3 "https://datasheet.lcsc.com/lcsc/1811021622_Samsung-Electro-Mechanics-CL10A105KP8NNNC_C26413.pdf" H 2600 6050 50  0001 C CNN
+F 3 "https://lcsc.com/product-detail/Multilayer-Ceramic-Capacitors-MLCC-SMD-SMT_Samsung-Electro-Mechanics-CL10A105KB8NNNC_C15849.html" H 2600 6050 50  0001 C CNN
 F 4 "Included in KiCad" H 2600 6050 50  0001 C CNN "3D-model"
-F 5 "https://lcsc.com/product-detail/Multilayer-Ceramic-Capacitors-MLCC-SMD-SMT_Samsung-Electro-Mechanics-CL10A105KP8NNNC_C26413.html" H 2600 6050 50  0001 C CNN "Link"
-F 6 "CL10A105KP8NNNC" H 2600 6050 50  0001 C CNN "MPN"
+F 5 "https://lcsc.com/product-detail/Multilayer-Ceramic-Capacitors-MLCC-SMD-SMT_Samsung-Electro-Mechanics-CL10A105KB8NNNC_C15849.html" H 2600 6050 50  0001 C CNN "Link"
+F 6 "CL10A105KB8NNNC" H 2600 6050 50  0001 C CNN "MPN"
 	1    2600 6050
 	1    0    0    -1
@@
 F 1 "1u X5R" V 10550 2750 50  0000 L CNN
 F 2 "Capacitor_SMD:C_0603_1608Metric" H 10438 2750 50  0001 C CNN
-F 3 "https://datasheet.lcsc.com/lcsc/1811021622_Samsung-Electro-Mechanics-CL10A105KP8NNNC_C26413.pdf" H 10400 2900 50  0001 C CNN
+F 3 "https://lcsc.com/product-detail/Multilayer-Ceramic-Capacitors-MLCC-SMD-SMT_Samsung-Electro-Mechanics-CL10A105KB8NNNC_C15849.html" H 10400 2900 50  0001 C CNN
 F 4 "Included in KiCad" H 10400 2900 50  0001 C CNN "3D-model"
-F 5 "https://lcsc.com/product-detail/Multilayer-Ceramic-Capacitors-MLCC-SMD-SMT_Samsung-Electro-Mechanics-CL10A105KP8NNNC_C26413.html" H 10400 2900 50  0001 C CNN "Link"
-F 6 "CL10A105KP8NNNC" H 10400 2900 50  0001 C CNN "MPN"
+F 5 "https://lcsc.com/product-detail/Multilayer-Ceramic-Capacitors-MLCC-SMD-SMT_Samsung-Electro-Mechanics-CL10A105KB8NNNC_C15849.html" H 10400 2900 50  0001 C CNN "Link"
+F 6 "CL10A105KB8NNNC" H 10400 2900 50  0001 C CNN "MPN"
 	1    10400 2900
 	0    -1   -1   0
@@
 F 1 "1u X5R" V 5300 3450 50  0000 L CNN
 F 2 "Capacitor_SMD:C_0603_1608Metric" H 5388 3250 50  0001 C CNN
-F 3 "https://datasheet.lcsc.com/lcsc/1811021622_Samsung-Electro-Mechanics-CL10A105KP8NNNC_C26413.pdf" H 5350 3400 50  0001 C CNN
+F 3 "https://lcsc.com/product-detail/Multilayer-Ceramic-Capacitors-MLCC-SMD-SMT_Samsung-Electro-Mechanics-CL10A105KB8NNNC_C15849.html" H 5350 3400 50  0001 C CNN
 F 4 "Included in KiCad" H 5350 3400 50  0001 C CNN "3D-model"
-F 5 "https://lcsc.com/product-detail/Multilayer-Ceramic-Capacitors-MLCC-SMD-SMT_Samsung-Electro-Mechanics-CL10A105KP8NNNC_C26413.html" H 5350 3400 50  0001 C CNN "Link"
-F 6 "CL10A105KP8NNNC" H 5350 3400 50  0001 C CNN "MPN"
+F 5 "https://lcsc.com/product-detail/Multilayer-Ceramic-Capacitors-MLCC-SMD-SMT_Samsung-Electro-Mechanics-CL10A105KB8NNNC_C15849.html" H 5350 3400 50  0001 C CNN "Link"
+F 6 "CL10A105KB8NNNC" H 5350 3400 50  0001 C CNN "MPN"
 	1    5350 3400
 	0    1    1    0
@@
 F 1 "1u X5R" H 8000 4750 50  0000 L CNN
 F 2 "Capacitor_SMD:C_0603_1608Metric" H 8138 4700 50  0001 C CNN
-F 3 "https://datasheet.lcsc.com/lcsc/1811021622_Samsung-Electro-Mechanics-CL10A105KP8NNNC_C26413.pdf" H 8100 4850 50  0001 C CNN
+F 3 "https://lcsc.com/product-detail/Multilayer-Ceramic-Capacitors-MLCC-SMD-SMT_Samsung-Electro-Mechanics-CL10A105KB8NNNC_C15849.html" H 8100 4850 50  0001 C CNN
 F 4 "Included in KiCad" H 8100 4850 50  0001 C CNN "3D-model"
-F 5 "https://lcsc.com/product-detail/Multilayer-Ceramic-Capacitors-MLCC-SMD-SMT_Samsung-Electro-Mechanics-CL10A105KP8NNNC_C26413.html" H 8100 4850 50  0001 C CNN "Link"
-F 6 "CL10A105KP8NNNC" H 8100 4850 50  0001 C CNN "MPN"
+F 5 "https://lcsc.com/product-detail/Multilayer-Ceramic-Capacitors-MLCC-SMD-SMT_Samsung-Electro-Mechanics-CL10A105KB8NNNC_C15849.html" H 8100 4850 50  0001 C CNN "Link"
+F 6 "CL10A105KB8NNNC" H 8100 4850 50  0001 C CNN "MPN"
 	1    8100 4850
 	1    0    0    -1

Commit message: production: 3n3 to 0603
Parts:
- C22: Link https://lcsc.com/product-detail/Multilayer-Ceramic-Capacitors-MLCC-SMD-SMT_CCTC-TCC0805X7R332K500DT_C282760.html -> https://lcsc.com/product-detail/Multilayer-Ceramic-Capacitors-MLCC-SMD-SMT_Samsung-Electro-Mechanics-CL10B332KB8NNNC_C1613.html; MPN TCC0805X7R332K500DT -> CL10B332KB8NNNC
Changed lines of the file:
@@
 F 1 "3n3 X7R" H 8550 3550 50  0000 L CNN
 F 2 "Capacitor_SMD:C_0603_1608Metric" H 8738 3500 50  0001 C CNN
-F 3 "https://datasheet.lcsc.com/szlcsc/1810181636_CCTC-TCC0805X7R332K500DT_C282760.pdf" H 8700 3650 50  0001 C CNN
+F 3 "https://datasheet.lcsc.com/lcsc/1810261513_Samsung-Electro-Mechanics-CL10B332KB8NNNC_C1613.pdf" H 8700 3650 50  0001 C CNN
 F 4 "Included in KiCad" H 8700 3650 50  0001 C CNN "3D-model"
-F 5 "https://lcsc.com/product-detail/Multilayer-Ceramic-Capacitors-MLCC-SMD-SMT_CCTC-TCC0805X7R332K500DT_C282760.html" H 8700 3650 50  0001 C CNN "Link"
-F 6 "TCC0805X7R332K500DT" H 8700 3650 50  0001 C CNN "MPN"
+F 5 "https://lcsc.com/product-detail/Multilayer-Ceramic-Capacitors-MLCC-SMD-SMT_Samsung-Electro-Mechanics-CL10B332KB8NNNC_C1613.html" H 8700 3650 50  0001 C CNN "Link"
+F 6 "CL10B332KB8NNNC" H 8700 3650 50  0001 C CNN "MPN"
 	1    8700 3650
 	1    0    0    -1
