File: osab.sch (KiCad schematic (older format))
At the start: 88 parts, among them CON1 TF-01A, CON2 PJ-3420-A-SMT, CON3 TYPE-C-31-M-12, Q1 BC847B, SW1 PPP, SW10 RESET, SW2 VOL-, SW3 VOL+, SW4 CHAP-, SW5 CHAP+, SW6 OT/NT, SW7 BOOK-, SW8 BOOK+, SW9 BUTTON_LOCK, U1 VS1000, U2 ME6211C33M5G-N, U3 25LC640A, U4 TP4055, U5 MF5853CS, U6 TCS7191, Y1 12MHz

Commit message: production: 47n to 0603
Parts:
- C19: Link https://lcsc.com/product-detail/Multilayer-Ceramic-Capacitors-MLCC-SMD-SMT_CCTC-TCC0805X7R473K500DT_C282770.html -> https://lcsc.com/product-detail/Multilayer-Ceramic-Capacitors-MLCC-SMD-SMT_Samsung-Electro-Mechanics-CL10B473KB8NNNC_C1622.html; MPN TCC0805X7R473K500DT -> CL10B473KB8NNNC
Changed lines of the file:
@@
 F 1 "47n X7R" H 7100 3900 50  0000 L CNN
 F 2 "Capacitor_SMD:C_0603_1608Metric" H 7488 3850 50  0001 C CNN
-F 3 "https://datasheet.lcsc.com/szlcsc/1810181648_CCTC-TCC0805X7R473K500DT_C282770.pdf" H 7450 4000 50  0001 C CNN
+F 3 "https://datasheet.lcsc.com/lcsc/1810261614_Samsung-Electro-Mechanics-CL10B473KB8NNNC_C1622.pdf" H 7450 4000 50  0001 C CNN
 F 4 "Included in KiCad" H 7450 4000 50  0001 C CNN "3D-model"
-F 5 "https://lcsc.com/product-detail/Multilayer-Ceramic-Capacitors-MLCC-SMD-SMT_CCTC-TCC0805X7R473K500DT_C282770.html" H 7450 4000 50  0001 C CNN "Link"
-F 6 "TCC0805X7R473K500DT" H 7450 4000 50  0001 C CNN "MPN"
+F 5 "https://lcsc.com/product-detail/Multilayer-Ceramic-Capacitors-MLCC-SMD-SMT_Samsung-Electro-Mechanics-CL10B473KB8NNNC_C1622.html" H 7450 4000 50  0001 C CNN "Link"
+F 6 "CL10B473KB8NNNC" H 7450 4000 50  0001 C CNN "MPN"
 	1    7450 4000
 	1    0    0    -1

Commit message: production: 10n to 0603
Parts:
- C20, C21: Link https://lcsc.com/product-detail/Multilayer-Ceramic-Capacitors-MLCC-SMD-SMT_SAMSUNG_CL21B103KBCNNNC_10nF-103-10-50V_C84715.html -> https://lcsc.com/product-detail/Multilayer-Ceramic-Capacitors-MLCC-SMD-SMT_Samsung-Electro-Mechanics-CL10B103KB8NNNC_C1589.html; MPN CL21B103KBCNNNC -> CL10B103KB8NNNC
Changed lines of the file:
@@
 F 1 "10n X7R" H 7500 3900 50  0000 L CNN
 F 2 "Capacitor_SMD:C_0603_1608Metric" H 7688 3850 50  0001 C CNN
-F 3 "https://datasheet.lcsc.com/szlcsc/1811122017_Samsung-Electro-Mechanics-CL21B103KBCNNNC_C84715.pdf" H 7650 4000 50  0001 C CNN
+F 3 "https://datasheet.lcsc.com/lcsc/1810191222_Samsung-Electro-Mechanics-CL10B103KB8NNNC_C1589.pdf" H 7650 4000 50  0001 C CNN
 F 4 "Included in KiCad" H 7650 4000 50  0001 C CNN "3D-model"
-F 5 "https://lcsc.com/product-detail/Multilayer-Ceramic-Capacitors-MLCC-SMD-SMT_SAMSUNG_CL21B103KBCNNNC_10nF-103-10-50V_C84715.html" H 7650 4000 50  0001 C CNN "Link"
-F 6 "CL21B103KBCNNNC" H 7650 4000 50  0001 C CNN "MPN"
+F 5 "https://lcsc.com/product-detail/Multilayer-Ceramic-Capacitors-MLCC-SMD-SMT_Samsung-Electro-Mechanics-CL10B103KB8NNNC_C1589.html" H 7650 4000 50  0001 C CNN "Link"
+F 6 "CL10B103KB8NNNC" H 7650 4000 50  0001 C CNN "MPN"
 	1    7650 4000
 	1    0    0    -1
@@
 F 1 "10n X7R" H 7850 3900 50  0000 L CNN
 F 2 "Capacitor_SMD:C_0603_1608Metric" H 7888 3850 50  0001 C CNN
-F 3 "https://datasheet.lcsc.com/szlcsc/1811122017_Samsung-Electro-Mechanics-CL21B103KBCNNNC_C84715.pdf" H 7850 4000 50  0001 C CNN
+F 3 "https://datasheet.lcsc.com/lcsc/1810191222_Samsung-Electro-Mechanics-CL10B103KB8NNNC_C1589.pdf" H 7850 4000 50  0001 C CNN
 F 4 "Included in KiCad" H 7850 4000 50  0001 C CNN "3D-model"
-F 5 "https://lcsc.com/product-detail/Multilayer-Ceramic-Capacitors-MLCC-SMD-SMT_SAMSUNG_CL21B103KBCNNNC_10nF-103-10-50V_C84715.html" H 7850 4000 50  0001 C CNN "Link"
-F 6 "CL21B103KBCNNNC" H 7850 4000 50  0001 C CNN "MPN"
+F 5 "https://lcsc.com/product-detail/Multilayer-Ceramic-Capacitors-MLCC-SMD-SMT_Samsung-Electro-Mechanics-CL10B103KB8NNNC_C1589.html" H 7850 4000 50  0001 C CNN "Link"
+F 6 "CL10B103KB8NNNC" H 7850 4000 50  0001 C CNN "MPN"
 	1    7850 4000
 	1    0    0    -1

Commit message: production: Changed all 0805 resistor footprints to 0603
Parts:
- R1, R10, R11, R12, R13, R14, R15, R16, R17, R18, R19, R2, R20, R21, R22, R23, R24, R25, R26, R27, R28, R29, R3, R30, R31, R32, R33, R34, R35, R36, R37, R4, R5, R6, R7, R8, R9: footprint Resistor_SMD:R_0805_2012Metric -> Resistor_SMD:R_0603_1608Metric

Commit message: production: Changed all 10k resistors to 0603
Parts:
- R11, R14, R2, R3, R31, R34, R4, R5, R6, R7, R8: Link https://lcsc.com/product-detail/Others_Viking-Tech-ARG05FTC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 -> https://lcsc.com/product-detail/Chip-Resistor-Surface-Mount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; MPN ARG05FTC1002 -> ARG03FTC1002
Changed lines of the file:
@@
 F 1 "10k" V 5050 1650 50  0000 C CNN
 F 2 "Resistor_SMD:R_0603_1608Metric" V 4980 1650 50  0001 C CNN
-F 3 "https://datasheet.lcsc.com/szlcsc/1810261818_Viking-Tech-ARG05FTC1002_C217770.pdf" H 5050 1650 50  0001 C CNN
+F 3 "https://datasheet.lcsc.com/lcsc/1811091612_Viking-Tech-ARG03FTC1002_C217687.pdf" H 5050 1650 50  0001 C CNN
 F 4 "Included in KiCad" H 5050 1650 50  0001 C CNN "3D-model"
-F 5 "https://lcsc.com/product-detail/Others_Viking-Tech-ARG05FTC1002_C217770.html" H 5050 1650 50  0001 C CNN "Link"
-F 6 "ARG05FTC1002" H 5050 1650 50  0001 C CNN "MPN"
+F 5 "https://lcsc.com/product-detail/Chip-Resistor-Surface-Mount_Viking-Tech-ARG03FTC1002_C217687.html" H 5050 1650 50  0001 C CNN "Link"
+F 6 "ARG03FTC1002" H 5050 1650 50  0001 C CNN "MPN"
 	1    5050 1650
 	0    1    1    0
@@
 F 1 "10k" V 1300 3450 50  0000 C CNN
 F 2 "Resistor_SMD:R_0603_1608Metric" V 1230 3450 50  0001 C CNN
-F 3 "https://datasheet.lcsc.com/szlcsc/1810261818_Viking-Tech-ARG05FTC1002_C217770.pdf" H 1300 3450 50  0001 C CNN
+F 3 "https://datasheet.lcsc.com/lcsc/1811091612_Viking-Tech-ARG03FTC1002_C217687.pdf" H 1300 3450 50  0001 C CNN
 F 4 "Included in KiCad" H 1300 3450 50  0001 C CNN "3D-model"
-F 5 "https://lcsc.com/product-detail/Others_Viking-Tech-ARG05FTC1002_C217770.html" H 1300 3450 50  0001 C CNN "Link"
-F 6 "ARG05FTC1002" H 1300 3450 50  0001 C CNN "MPN"
+F 5 "https://lcsc.com/product-detail/Chip-Resistor-Surface-Mount_Viking-Tech-ARG03FTC1002_C217687.html" H 1300 3450 50  0001 C CNN "Link"
+F 6 "ARG03FTC1002" H 1300 3450 50  0001 C CNN "MPN"
 	1    1300 3450
 	1    0    0    -1
@@
 F 1 "10k" V 1500 3450 50  0000 C CNN
 F 2 "Resistor_SMD:R_0603_1608Metric" V 1430 3450 50  0001 C CNN
-F 3 "https://datasheet.lcsc.com/szlcsc/1810261818_Viking-Tech-ARG05FTC1002_C217770.pdf" H 1500 3450 50  0001 C CNN
+F 3 "https://datasheet.lcsc.com/lcsc/1811091612_Viking-Tech-ARG03FTC1002_C217687.pdf" H 1500 3450 50  0001 C CNN
 F 4 "Included in KiCad" H 1500 3450 50  0001 C CNN "3D-model"
-F 5 "https://lcsc.com/product-detail/Others_Viking-Tech-ARG05FTC1002_C217770.html" H 1500 3450 50  0001 C CNN "Link"
-F 6 "ARG05FTC1002" H 1500 3450 50  0001 C CNN "MPN"
+F 5 "https://lcsc.com/product-detail/Chip-Resistor-Surface-Mount_Viking-Tech-ARG03FTC1002_C217687.html" H 1500 3450 50  0001 C CNN "Link"
+F 6 "ARG03FTC1002" H 1500 3450 50  0001 C CNN "MPN"
 	1    1500 3450
 	1    0    0    -1
@@
 F 1 "10k" V 1700 3450 50  0000 C CNN
 F 2 "Resistor_SMD:R_0603_1608Metric" V 1630 3450 50  0001 C CNN
-F 3 "https://datasheet.lcsc.com/szlcsc/1810261818_Viking-Tech-ARG05FTC1002_C217770.pdf" H 1700 3450 50  0001 C CNN
+F 3 "https://datasheet.lcsc.com/lcsc/1811091612_Viking-Tech-ARG03FTC1002_C217687.pdf" H 1700 3450 50  0001 C CNN
 F 4 "Included in KiCad" H 1700 3450 50  0001 C CNN "3D-model"
-F 5 "https://lcsc.com/product-detail/Others_Viking-Tech-ARG05FTC1002_C217770.html" H 1700 3450 50  0001 C CNN "Link"
-F 6 "ARG05FTC1002" H 1700 3450 50  0001 C CNN "MPN"
+F 5 "https://lcsc.com/product-detail/Chip-Resistor-Surface-Mount_Viking-Tech-ARG03FTC1002_C217687.html" H 1700 3450 50  0001 C CNN "Link"
+F 6 "ARG03FTC1002" H 1700 3450 50  0001 C CNN "MPN"
 	1    1700 3450
 	1    0    0    -1
@@
 F 1 "10k" V 1900 3450 50  0000 C CNN
 F 2 "Resistor_SMD:R_0603_1608Metric" V 1830 3450 50  0001 C CNN
-F 3 "https://datasheet.lcsc.com/szlcsc/1810261818_Viking-Tech-ARG05FTC1002_C217770.pdf" H 1900 3450 50  0001 C CNN
+F 3 "https://datasheet.lcsc.com/lcsc/1811091612_Viking-Tech-ARG03FTC1002_C217687.pdf" H 1900 3450 50  0001 C CNN
 F 4 "Included in KiCad" H 1900 3450 50  0001 C CNN "3D-model"
-F 5 "https://lcsc.com/product-detail/Others_Viking-Tech-ARG05FTC1002_C217770.html" H 1900 3450 50  0001 C CNN "Link"
-F 6 "ARG05FTC1002" H 1900 3450 50  0001 C CNN "MPN"
+F 5 "https://lcsc.com/product-detail/Chip-Resistor-Surface-Mount_Viking-Tech-ARG03FTC1002_C217687.html" H 1900 3450 50  0001 C CNN "Link"
+F 6 "ARG03FTC1002" H 1900 3450 50  0001 C CNN "MPN"
 	1    1900 3450
 	1    0    0    -1
@@
 F 1 "10k" V 2100 3450 50  0000 C CNN
 F 2 "Resistor_SMD:R_0603_1608Metric" V 2030 3450 50  0001 C CNN
-F 3 "https://datasheet.lcsc.com/szlcsc/1810261818_Viking-Tech-ARG05FTC1002_C217770.pdf" H 2100 3450 50  0001 C CNN
+F 3 "https://datasheet.lcsc.com/lcsc/1811091612_Viking-Tech-ARG03FTC1002_C217687.pdf" H 2100 3450 50  0001 C CNN
 F 4 "Included in KiCad" H 2100 3450 50  0001 C CNN "3D-model"
-F 5 "https://lcsc.com/product-detail/Others_Viking-Tech-ARG05FTC1002_C217770.html" H 2100 3450 50  0001 C CNN "Link"
-F 6 "ARG05FTC1002" H 2100 3450 50  0001 C CNN "MPN"
+F 5 "https://lcsc.com/product-detail/Chip-Resistor-Surface-Mount_Viking-Tech-ARG03FTC1002_C217687.html" H 2100 3450 50  0001 C CNN "Link"
+F 6 "ARG03FTC1002" H 2100 3450 50  0001 C CNN "MPN"
 	1    2100 3450
 	1    0    0    -1
@@
 F 1 "10k" V 2300 3450 50  0000 C CNN
 F 2 "Resistor_SMD:R_0603_1608Metric" V 2230 3450 50  0001 C CNN
-F 3 "https://datasheet.lcsc.com/szlcsc/1810261818_Viking-Tech-ARG05FTC1002_C217770.pdf" H 2300 3450 50  0001 C CNN
+F 3 "https://datasheet.lcsc.com/lcsc/1811091612_Viking-Tech-ARG03FTC1002_C217687.pdf" H 2300 3450 50  0001 C CNN
 F 4 "Included in KiCad" H 2300 3450 50  0001 C CNN "3D-model"
-F 5 "https://lcsc.com/product-detail/Others_Viking-Tech-ARG05FTC1002_C217770.html" H 2300 3450 50  0001 C CNN "Link"
-F 6 "ARG05FTC1002" H 2300 3450 50  0001 C CNN "MPN"
+F 5 "https://lcsc.com/product-detail/Chip-Resistor-Surface-Mount_Viking-Tech-ARG03FTC1002_C217687.html" H 2300 3450 50  0001 C CNN "Link"
+F 6 "ARG03FTC1002" H 2300 3450 50  0001 C CNN "MPN"
 	1    2300 3450
 	1    0    0    -1
@@
 F 1 "10k" V 2500 3450 50  0000 C CNN
 F 2 "Resistor_SMD:R_0603_1608Metric" V 2430 3450 50  0001 C CNN
-F 3 "https://datasheet.lcsc.com/szlcsc/1810261818_Viking-Tech-ARG05FTC1002_C217770.pdf" H 2500 3450 50  0001 C CNN
+F 3 "https://datasheet.lcsc.com/lcsc/1811091612_Viking-Tech-ARG03FTC1002_C217687.pdf" H 2500 3450 50  0001 C CNN
 F 4 "Included in KiCad" H 2500 3450 50  0001 C CNN "3D-model"
-F 5 "https://lcsc.com/product-detail/Others_Viking-Tech-ARG05FTC1002_C217770.html" H 2500 3450 50  0001 C CNN "Link"
-F 6 "ARG05FTC1002" H 2500 3450 50  0001 C CNN "MPN"
+F 5 "https://lcsc.com/product-detail/Chip-Resistor-Surface-Mount_Viking-Tech-ARG03FTC1002_C217687.html" H 2500 3450 50  0001 C CNN "Link"
+F 6 "ARG03FTC1002" H 2500 3450 50  0001 C CNN "MPN"
 	1    2500 3450
 	1    0    0    -1
@@
 F 1 "10k" V 2250 5100 50  0000 C CNN
 F 2 "Resistor_SMD:R_0603_1608Metric" V 2180 5100 50  0001 C CNN
-F 3 "https://datasheet.lcsc.com/szlcsc/1810261818_Viking-Tech-ARG05FTC1002_C217770.pdf" H 2250 5100 50  0001 C CNN
+F 3 "https://datasheet.lcsc.com/lcsc/1811091612_Viking-Tech-ARG03FTC1002_C217687.pdf" H 2250 5100 50  0001 C CNN
 F 4 "Included in KiCad" H 2250 5100 50  0001 C CNN "3D-model"
-F 5 "https://lcsc.com/product-detail/Others_Viking-Tech-ARG05FTC1002_C217770.html" H 2250 5100 50  0001 C CNN "Link"
-F 6 "ARG05FTC1002" H 2250 5100 50  0001 C CNN "MPN"
+F 5 "https://lcsc.com/product-detail/Chip-Resistor-Surface-Mount_Viking-Tech-ARG03FTC1002_C217687.html" H 2250 5100 50  0001 C CNN "Link"
+F 6 "ARG03FTC1002" H 2250 5100 50  0001 C CNN "MPN"
 	1    2250 5100
 	0    1    1    0
@@
 F 1 "10k" V 8700 2900 50  0000 C CNN
 F 2 "Resistor_SMD:R_0603_1608Metric" V 8630 2900 50  0001 C CNN
-F 3 "https://datasheet.lcsc.com/szlcsc/1810261818_Viking-Tech-ARG05FTC1002_C217770.pdf" H 8700 2900 50  0001 C CNN
+F 3 "https://datasheet.lcsc.com/lcsc/1811091612_Viking-Tech-ARG03FTC1002_C217687.pdf" H 8700 2900 50  0001 C CNN
 F 4 "Included in KiCad" H 8700 2900 50  0001 C CNN "3D-model"
-F 5 "https://lcsc.com/product-detail/Others_Viking-Tech-ARG05FTC1002_C217770.html" H 8700 2900 50  0001 C CNN "Link"
-F 6 "ARG05FTC1002" H 8700 2900 50  0001 C CNN "MPN"
+F 5 "https://lcsc.com/product-detail/Chip-Resistor-Surface-Mount_Viking-Tech-ARG03FTC1002_C217687.html" H 8700 2900 50  0001 C CNN "Link"
+F 6 "ARG03FTC1002" H 8700 2900 50  0001 C CNN "MPN"
 	1    8700 2900
 	1    0    0    -1
@@
 F 1 "10k" V 850 3500 50  0000 C CNN
 F 2 "Resistor_SMD:R_0603_1608Metric" V 780 3500 50  0001 C CNN
-F 3 "https://datasheet.lcsc.com/szlcsc/1810261818_Viking-Tech-ARG05FTC1002_C217770.pdf" H 850 3500 50  0001 C CNN
+F 3 "https://datasheet.lcsc.com/lcsc/1811091612_Viking-Tech-ARG03FTC1002_C217687.pdf" H 850 3500 50  0001 C CNN
 F 4 "Included in KiCad" H 850 3500 50  0001 C CNN "3D-model"
-F 5 "https://lcsc.com/product-detail/Others_Viking-Tech-ARG05FTC1002_C217770.html" H 850 3500 50  0001 C CNN "Link"
-F 6 "ARG05FTC1002" H 850 3500 50  0001 C CNN "MPN"
+F 5 "https://lcsc.com/product-detail/Chip-Resistor-Surface-Mount_Viking-Tech-ARG03FTC1002_C217687.html" H 850 3500 50  0001 C CNN "Link"
+F 6 "ARG03FTC1002" H 850 3500 50  0001 C CNN "MPN"
 	1    850  3500
 	1    0    0    -1

Commit message: production: Changed all 100k resistors to 0603
Parts:
- R1, R10, R12, R15, R16, R17, R18, R19, R22: Link https://lcsc.com/product-detail/Others_Viking-Tech-ARG05FTC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 -> https://lcsc.com/product-detail/Chip-Resistor-Surface-Mount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; MPN ARG05FTC1003 -> ARG03FTC1003
Changed lines of the file:
@@
 F 1 "100k" V 5550 1650 50  0000 C CNN
 F 2 "Resistor_SMD:R_0603_1608Metric" V 5480 1650 50  0001 C CNN
-F 3 "https://datasheet.lcsc.com/szlcsc/1810261818_Viking-Tech-ARG05FTC1003_C217765.pdf" H 5550 1650 50  0001 C CNN
+F 3 "https://datasheet.lcsc.com/lcsc/1811091512_Viking-Tech-ARG03FTC1003_C217682.pdf" H 5550 1650 50  0001 C CNN
 F 4 "Included in KiCad" H 5550 1650 50  0001 C CNN "3D-model"
-F 5 "https://lcsc.com/product-detail/Others_Viking-Tech-ARG05FTC1003_C217765.html" H 5550 1650 50  0001 C CNN "Link"
-F 6 "ARG05FTC1003" H 5550 1650 50  0001 C CNN "MPN"
+F 5 "https://lcsc.com/product-detail/Chip-Resistor-Surface-Mount_Viking-Tech-ARG03FTC1003_C217682.html" H 5550 1650 50  0001 C CNN "Link"
+F 6 "ARG03FTC1003" H 5550 1650 50  0001 C CNN "MPN"
 	1    5550 1650
 	0    1    1    0
@@
 F 1 "100k" V 3400 1200 50  0000 C CNN
 F 2 "Resistor_SMD:R_0603_1608Metric" V 3330 1200 50  0001 C CNN
-F 3 "https://datasheet.lcsc.com/szlcsc/1810261818_Viking-Tech-ARG05FTC1003_C217765.pdf" H 3400 1200 50  0001 C CNN
+F 3 "https://datasheet.lcsc.com/lcsc/1811091512_Viking-Tech-ARG03FTC1003_C217682.pdf" H 3400 1200 50  0001 C CNN
 F 4 "Included in KiCad" H 3400 1200 50  0001 C CNN "3D-model"
-F 5 "https://lcsc.com/product-detail/Others_Viking-Tech-ARG05FTC1003_C217765.html" H 3400 1200 50  0001 C CNN "Link"
-F 6 "ARG05FTC1003" H 3400 1200 50  0001 C CNN "MPN"
+F 5 "https://lcsc.com/product-detail/Chip-Resistor-Surface-Mount_Viking-Tech-ARG03FTC1003_C217682.html" H 3400 1200 50  0001 C CNN "Link"
+F 6 "ARG03FTC1003" H 3400 1200 50  0001 C CNN "MPN"
 	1    3400 1200
 	1    0    0    -1
@@
 F 1 "100k" V 850 2250 50  0000 C CNN
 F 2 "Resistor_SMD:R_0603_1608Metric" V 780 2250 50  0001 C CNN
-F 3 "https://datasheet.lcsc.com/szlcsc/1810261818_Viking-Tech-ARG05FTC1003_C217765.pdf" H 850 2250 50  0001 C CNN
+F 3 "https://datasheet.lcsc.com/lcsc/1811091512_Viking-Tech-ARG03FTC1003_C217682.pdf" H 850 2250 50  0001 C CNN
 F 4 "Included in KiCad" H 850 2250 50  0001 C CNN "3D-model"
-F 5 "https://lcsc.com/product-detail/Others_Viking-Tech-ARG05FTC1003_C217765.html" H 850 2250 50  0001 C CNN "Link"
-F 6 "ARG05FTC1003" H 850 2250 50  0001 C CNN "MPN"
+F 5 "https://lcsc.com/product-detail/Chip-Resistor-Surface-Mount_Viking-Tech-ARG03FTC1003_C217682.html" H 850 2250 50  0001 C CNN "Link"
+F 6 "ARG03FTC1003" H 850 2250 50  0001 C CNN "MPN"
 	1    850  2250
 	1    0    0    -1
@@
 F 1 "100k" V 2650 4000 50  0000 C CNN
 F 2 "Resistor_SMD:R_0603_1608Metric" V 2580 4000 50  0001 C CNN
-F 3 "https://datasheet.lcsc.com/szlcsc/1810261818_Viking-Tech-ARG05FTC1003_C217765.pdf" H 2650 4000 50  0001 C CNN
+F 3 "https://datasheet.lcsc.com/lcsc/1811091512_Viking-Tech-ARG03FTC1003_C217682.pdf" H 2650 4000 50  0001 C CNN
 F 4 "Included in KiCad" H 2650 4000 50  0001 C CNN "3D-model"
-F 5 "https://lcsc.com/product-detail/Others_Viking-Tech-ARG05FTC1003_C217765.html" H 2650 4000 50  0001 C CNN "Link"
-F 6 "ARG05FTC1003" H 2650 4000 50  0001 C CNN "MPN"
+F 5 "https://lcsc.com/product-detail/Chip-Resistor-Surface-Mount_Viking-Tech-ARG03FTC1003_C217682.html" H 2650 4000 50  0001 C CNN "Link"
+F 6 "ARG03FTC1003" H 2650 4000 50  0001 C CNN "MPN"
 	1    2650 4000
 	0    1    1    0
@@
 F 1 "100k" V 5400 4050 50  0000 C CNN
 F 2 "Resistor_SMD:R_0603_1608Metric" V 5330 4050 50  0001 C CNN
-F 3 "https://datasheet.lcsc.com/szlcsc/1810261818_Viking-Tech-ARG05FTC1003_C217765.pdf" H 5400 4050 50  0001 C CNN
+F 3 "https://datasheet.lcsc.com/lcsc/1811091512_Viking-Tech-ARG03FTC1003_C217682.pdf" H 5400 4050 50  0001 C CNN
 F 4 "Included in KiCad" H 5400 4050 50  0001 C CNN "3D-model"
-F 5 "https://lcsc.com/product-detail/Others_Viking-Tech-ARG05FTC1003_C217765.html" H 5400 4050 50  0001 C CNN "Link"
-F 6 "ARG05FTC1003" H 5400 4050 50  0001 C CNN "MPN"
+F 5 "https://lcsc.com/product-detail/Chip-Resistor-Surface-Mount_Viking-Tech-ARG03FTC1003_C217682.html" H 5400 4050 50  0001 C CNN "Link"
+F 6 "ARG03FTC1003" H 5400 4050 50  0001 C CNN "MPN"
 	1    5400 4050
 	0    1    1    0
@@
 F 1 "100k" V 5400 4450 50  0000 C CNN
 F 2 "Resistor_SMD:R_0603_1608Metric" V 5330 4450 50  0001 C CNN
-F 3 "https://datasheet.lcsc.com/szlcsc/1810261818_Viking-Tech-ARG05FTC1003_C217765.pdf" H 5400 4450 50  0001 C CNN
+F 3 "https://datasheet.lcsc.com/lcsc/1811091512_Viking-Tech-ARG03FTC1003_C217682.pdf" H 5400 4450 50  0001 C CNN
 F 4 "Included in KiCad" H 5400 4450 50  0001 C CNN "3D-model"
-F 5 "https://lcsc.com/product-detail/Others_Viking-Tech-ARG05FTC1003_C217765.html" H 5400 4450 50  0001 C CNN "Link"
-F 6 "ARG05FTC1003" H 5400 4450 50  0001 C CNN "MPN"
+F 5 "https://lcsc.com/product-detail/Chip-Resistor-Surface-Mount_Viking-Tech-ARG03FTC1003_C217682.html" H 5400 4450 50  0001 C CNN "Link"
+F 6 "ARG03FTC1003" H 5400 4450 50  0001 C CNN "MPN"
 	1    5400 4450
 	0    1    1    0
@@
 F 1 "100k" V 5400 4550 50  0000 C CNN
 F 2 "Resistor_SMD:R_0603_1608Metric" V 5330 4550 50  0001 C CNN
-F 3 "https://datasheet.lcsc.com/szlcsc/1810261818_Viking-Tech-ARG05FTC1003_C217765.pdf" H 5400 4550 50  0001 C CNN
+F 3 "https://datasheet.lcsc.com/lcsc/1811091512_Viking-Tech-ARG03FTC1003_C217682.pdf" H 5400 4550 50  0001 C CNN
 F 4 "Included in KiCad" H 5400 4550 50  0001 C CNN "3D-model"
-F 5 "https://lcsc.com/product-detail/Others_Viking-Tech-ARG05FTC1003_C217765.html" H 5400 4550 50  0001 C CNN "Link"
-F 6 "ARG05FTC1003" H 5400 4550 50  0001 C CNN "MPN"
+F 5 "https://lcsc.com/product-detail/Chip-Resistor-Surface-Mount_Viking-Tech-ARG03FTC1003_C217682.html" H 5400 4550 50  0001 C CNN "Link"
+F 6 "ARG03FTC1003" H 5400 4550 50  0001 C CNN "MPN"
 	1    5400 4550
 	0    1    1    0
@@
 F 1 "100k" V 7000 3600 50  0000 C CNN
 F 2 "Resistor_SMD:R_0603_1608Metric" V 6930 3600 50  0001 C CNN
-F 3 "https://datasheet.lcsc.com/szlcsc/1810261818_Viking-Tech-ARG05FTC1003_C217765.pdf" H 7000 3600 50  0001 C CNN
+F 3 "https://datasheet.lcsc.com/lcsc/1811091512_Viking-Tech-ARG03FTC1003_C217682.pdf" H 7000 3600 50  0001 C CNN
 F 4 "Included in KiCad" H 7000 3600 50  0001 C CNN "3D-model"
-F 5 "https://lcsc.com/product-detail/Others_Viking-Tech-ARG05FTC1003_C217765.html" H 7000 3600 50  0001 C CNN "Link"
-F 6 "ARG05FTC1003" H 7000 3600 50  0001 C CNN "MPN"
+F 5 "https://lcsc.com/product-detail/Chip-Resistor-Surface-Mount_Viking-Tech-ARG03FTC1003_C217682.html" H 7000 3600 50  0001 C CNN "Link"
+F 6 "ARG03FTC1003" H 7000 3600 50  0001 C CNN "MPN"
 	1    7000 3600
 	0    1    1    0
@@
 F 1 "100k" V 9300 4050 50  0000 C CNN
 F 2 "Resistor_SMD:R_0603_1608Metric" V 9230 4050 50  0001 C CNN
-F 3 "https://datasheet.lcsc.com/szlcsc/1810261818_Viking-Tech-ARG05FTC1003_C217765.pdf" H 9300 4050 50  0001 C CNN
+F 3 "https://datasheet.lcsc.com/lcsc/1811091512_Viking-Tech-ARG03FTC1003_C217682.pdf" H 9300 4050 50  0001 C CNN
 F 4 "Included in KiCad" H 9300 4050 50  0001 C CNN "3D-model"
-F 5 "https://lcsc.com/product-detail/Others_Viking-Tech-ARG05FTC1003_C217765.html" H 9300 4050 50  0001 C CNN "Link"
-F 6 "ARG05FTC1003" H 9300 4050 50  0001 C CNN "MPN"
+F 5 "https://lcsc.com/product-detail/Chip-Resistor-Surface-Mount_Viking-Tech-ARG03FTC1003_C217682.html" H 9300 4050 50  0001 C CNN "Link"
+F 6 "ARG03FTC1003" H 9300 4050 50  0001 C CNN "MPN"
 	1    9300 4050
 	1    0    0    -1

Commit message: production: Changed 1m resistor to 0603
Parts:
- R9: Link https://lcsc.com/product-detail/Others_Viking-Tech-ARG05FTC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 -> https://lcsc.com/product-detail/Chip-Resistor-Surface-Mount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; MPN ARG05FTC1004 -> AR03FTC1004
Changed lines of the file:
@@
 F 1 "1m" V 2750 1650 50  0000 C CNN
 F 2 "Resistor_SMD:R_0603_1608Metric" V 2680 1650 50  0001 C CNN
-F 3 "https://datasheet.lcsc.com/szlcsc/1810261826_Viking-Tech-ARG05FTC1004_C218408.pdf" H 2750 1650 50  0001 C CNN
+F 3 "https://datasheet.lcsc.com/lcsc/1912111437_Viking-Tech-AR03FTC1004_C234360.pdf" H 2750 1650 50  0001 C CNN
 F 4 "Included in KiCad" H 2750 1650 50  0001 C CNN "3D-model"
-F 5 "https://lcsc.com/product-detail/Others_Viking-Tech-ARG05FTC1004_C218408.html" H 2750 1650 50  0001 C CNN "Link"
-F 6 "ARG05FTC1004" H 2750 1650 50  0001 C CNN "MPN"
+F 5 "https://lcsc.com/product-detail/Chip-Resistor-Surface-Mount_Viking-Tech-AR03FTC1004_C234360.html" H 2750 1650 50  0001 C CNN "Link"
+F 6 "AR03FTC1004" H 2750 1650 50  0001 C CNN "MPN"
 	1    2750 1650
 	0    1    1    0
