File: osab.sch (KiCad schematic (older format))
At the start: 88 parts, among them CON1 TF-01A, CON2 PJ-3420-A-SMT, CON3 TYPE-C-31-M-12, Q1 BC847B, SW1 PPP, SW10 RESET, SW2 VOL-, SW3 VOL+, SW4 CHAP-, SW5 CHAP+, SW6 OT/NT, SW7 BOOK-, SW8 BOOK+, SW9 BUTTON_LOCK, U1 VS1000, U2 ME6211C33M5G-N, U3 25LC640A, U4 TP4055, U5 MF5853CS, U6 TCS7191, Y1 12MHz

Commit message: production: Changed all 1k resistors to 0603
Parts:
- R13, R20, R30, R32, R35: Link https://lcsc.com/product-detail/Others_Viking-Tech-ARG05FTC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 -> https://lcsc.com/product-detail/Chip-Resistor-Surface-Mount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; MPN ARG05FTC1001 -> ARG03FTC1001
Changed lines of the file:
@@
 F 1 "1k" V 2650 4200 50  0000 C CNN
 F 2 "Resistor_SMD:R_0603_1608Metric" V 2580 4200 50  0001 C CNN
-F 3 "https://datasheet.lcsc.com/szlcsc/1811111513_Viking-Tech-ARG05FTC1001_C218388.pdf" H 2650 4200 50  0001 C CNN
+F 3 "https://datasheet.lcsc.com/lcsc/1811111521_Viking-Tech-ARG03FTC1001_C217840.pdf" H 2650 4200 50  0001 C CNN
 F 4 "Included in KiCad" H 2650 4200 50  0001 C CNN "3D-model"
-F 5 "https://lcsc.com/product-detail/Others_Viking-Tech-ARG05FTC1001_C218388.html" H 2650 4200 50  0001 C CNN "Link"
-F 6 "ARG05FTC1001" H 2650 4200 50  0001 C CNN "MPN"
+F 5 "https://lcsc.com/product-detail/Chip-Resistor-Surface-Mount_Viking-Tech-ARG03FTC1001_C217840.html" H 2650 4200 50  0001 C CNN "Link"
+F 6 "ARG03FTC1001" H 2650 4200 50  0001 C CNN "MPN"
 	1    2650 4200
 	0    1    1    0
@@
 F 1 "1k" V 8700 2400 50  0000 C CNN
 F 2 "Resistor_SMD:R_0603_1608Metric" V 8630 2400 50  0001 C CNN
-F 3 "https://datasheet.lcsc.com/szlcsc/1811111513_Viking-Tech-ARG05FTC1001_C218388.pdf" H 8700 2400 50  0001 C CNN
+F 3 "https://datasheet.lcsc.com/lcsc/1811111521_Viking-Tech-ARG03FTC1001_C217840.pdf" H 8700 2400 50  0001 C CNN
 F 4 "Included in KiCad" H 8700 2400 50  0001 C CNN "3D-model"
-F 5 "https://lcsc.com/product-detail/Others_Viking-Tech-ARG05FTC1001_C218388.html" H 8700 2400 50  0001 C CNN "Link"
-F 6 "ARG05FTC1001" H 8700 2400 50  0001 C CNN "MPN"
+F 5 "https://lcsc.com/product-detail/Chip-Resistor-Surface-Mount_Viking-Tech-ARG03FTC1001_C217840.html" H 8700 2400 50  0001 C CNN "Link"
+F 6 "ARG03FTC1001" H 8700 2400 50  0001 C CNN "MPN"
 	1    8700 2400
 	1    0    0    -1
@@
 F 1 "1k" V 9250 2450 50  0000 C CNN
 F 2 "Resistor_SMD:R_0603_1608Metric" V 9180 2450 50  0001 C CNN
-F 3 "https://datasheet.lcsc.com/szlcsc/1811111513_Viking-Tech-ARG05FTC1001_C218388.pdf" H 9250 2450 50  0001 C CNN
+F 3 "https://datasheet.lcsc.com/lcsc/1811111521_Viking-Tech-ARG03FTC1001_C217840.pdf" H 9250 2450 50  0001 C CNN
 F 4 "Included in KiCad" H 9250 2450 50  0001 C CNN "3D-model"
-F 5 "https://lcsc.com/product-detail/Others_Viking-Tech-ARG05FTC1001_C218388.html" H 9250 2450 50  0001 C CNN "Link"
-F 6 "ARG05FTC1001" H 9250 2450 50  0001 C CNN "MPN"
+F 5 "https://lcsc.com/product-detail/Chip-Resistor-Surface-Mount_Viking-Tech-ARG03FTC1001_C217840.html" H 9250 2450 50  0001 C CNN "Link"
+F 6 "ARG03FTC1001" H 9250 2450 50  0001 C CNN "MPN"
 	1    9250 2450
 	0    1    1    0
@@
 F 1 "1k" V 8700 4800 50  0000 C CNN
 F 2 "Resistor_SMD:R_0603_1608Metric" V 8630 4800 50  0001 C CNN
-F 3 "https://datasheet.lcsc.com/szlcsc/1811111513_Viking-Tech-ARG05FTC1001_C218388.pdf" H 8700 4800 50  0001 C CNN
+F 3 "https://datasheet.lcsc.com/lcsc/1811111521_Viking-Tech-ARG03FTC1001_C217840.pdf" H 8700 4800 50  0001 C CNN
 F 4 "Included in KiCad" H 8700 4800 50  0001 C CNN "3D-model"
-F 5 "https://lcsc.com/product-detail/Others_Viking-Tech-ARG05FTC1001_C218388.html" H 8700 4800 50  0001 C CNN "Link"
-F 6 "ARG05FTC1001" H 8700 4800 50  0001 C CNN "MPN"
+F 5 "https://lcsc.com/product-detail/Chip-Resistor-Surface-Mount_Viking-Tech-ARG03FTC1001_C217840.html" H 8700 4800 50  0001 C CNN "Link"
+F 6 "ARG03FTC1001" H 8700 4800 50  0001 C CNN "MPN"
 	1    8700 4800
 	0    1    1    0
@@
 F 1 "1k" V 2000 1550 50  0000 C CNN
 F 2 "Resistor_SMD:R_0603_1608Metric" V 1930 1550 50  0001 C CNN
-F 3 "https://datasheet.lcsc.com/szlcsc/1811111513_Viking-Tech-ARG05FTC1001_C218388.pdf" H 2000 1550 50  0001 C CNN
+F 3 "https://datasheet.lcsc.com/lcsc/1811111521_Viking-Tech-ARG03FTC1001_C217840.pdf" H 2000 1550 50  0001 C CNN
 F 4 "Included in KiCad" H 2000 1550 50  0001 C CNN "3D-model"
-F 5 "https://lcsc.com/product-detail/Others_Viking-Tech-ARG05FTC1001_C218388.html" H 2000 1550 50  0001 C CNN "Link"
-F 6 "ARG05FTC1001" H 2000 1550 50  0001 C CNN "MPN"
+F 5 "https://lcsc.com/product-detail/Chip-Resistor-Surface-Mount_Viking-Tech-ARG03FTC1001_C217840.html" H 2000 1550 50  0001 C CNN "Link"
+F 6 "ARG03FTC1001" H 2000 1550 50  0001 C CNN "MPN"
 	1    2000 1550
 	1    0    0    -1

Commit message: production: Changed all 10R resistors to 0603
Parts:
- R23, R26, R27: Link https://lcsc.com/product-detail/Others_Viking-Tech-ARG05FTC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 -> https://lcsc.com/product-detail/Chip-Resistor-Surface-Mount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; MPN ARG05FTC0100 -> ARG03FTC0100
Changed lines of the file:
@@
 F 1 "10" V 7450 3650 50  0000 C CNN
 F 2 "Resistor_SMD:R_0603_1608Metric" V 7380 3650 50  0001 C CNN
-F 3 "https://datasheet.lcsc.com/szlcsc/1810261818_Viking-Tech-ARG05FTC0100_C217774.pdf" H 7450 3650 50  0001 C CNN
+F 3 "https://datasheet.lcsc.com/lcsc/1811111520_Viking-Tech-ARG03FTC0100_C217691.pdf" H 7450 3650 50  0001 C CNN
 F 4 "Included in KiCad" H 7450 3650 50  0001 C CNN "3D-model"
-F 5 "https://lcsc.com/product-detail/Others_Viking-Tech-ARG05FTC0100_C217774.html" H 7450 3650 50  0001 C CNN "Link"
-F 6 "ARG05FTC0100" H 7450 3650 50  0001 C CNN "MPN"
+F 5 "https://lcsc.com/product-detail/Chip-Resistor-Surface-Mount_Viking-Tech-ARG03FTC0100_C217691.html" H 7450 3650 50  0001 C CNN "Link"
+F 6 "ARG03FTC0100" H 7450 3650 50  0001 C CNN "MPN"
 	1    7450 3650
 	-1   0    0    1
@@
 F 1 "10" V 8200 3000 50  0000 C CNN
 F 2 "Resistor_SMD:R_0603_1608Metric" V 8130 3000 50  0001 C CNN
-F 3 "https://datasheet.lcsc.com/szlcsc/1810261818_Viking-Tech-ARG05FTC0100_C217774.pdf" H 8200 3000 50  0001 C CNN
+F 3 "https://datasheet.lcsc.com/lcsc/1811111520_Viking-Tech-ARG03FTC0100_C217691.pdf" H 8200 3000 50  0001 C CNN
 F 4 "Included in KiCad" H 8200 3000 50  0001 C CNN "3D-model"
-F 5 "https://lcsc.com/product-detail/Others_Viking-Tech-ARG05FTC0100_C217774.html" H 8200 3000 50  0001 C CNN "Link"
-F 6 "ARG05FTC0100" H 8200 3000 50  0001 C CNN "MPN"
+F 5 "https://lcsc.com/product-detail/Chip-Resistor-Surface-Mount_Viking-Tech-ARG03FTC0100_C217691.html" H 8200 3000 50  0001 C CNN "Link"
+F 6 "ARG03FTC0100" H 8200 3000 50  0001 C CNN "MPN"
 	1    8200 3000
 	0    -1   -1   0
@@
 F 1 "10" V 8400 3100 50  0000 C CNN
 F 2 "Resistor_SMD:R_0603_1608Metric" V 8330 3100 50  0001 C CNN
-F 3 "https://datasheet.lcsc.com/szlcsc/1810261818_Viking-Tech-ARG05FTC0100_C217774.pdf" H 8400 3100 50  0001 C CNN
+F 3 "https://datasheet.lcsc.com/lcsc/1811111520_Viking-Tech-ARG03FTC0100_C217691.pdf" H 8400 3100 50  0001 C CNN
 F 4 "Included in KiCad" H 8400 3100 50  0001 C CNN "3D-model"
-F 5 "https://lcsc.com/product-detail/Others_Viking-Tech-ARG05FTC0100_C217774.html" H 8400 3100 50  0001 C CNN "Link"
-F 6 "ARG05FTC0100" H 8400 3100 50  0001 C CNN "MPN"
+F 5 "https://lcsc.com/product-detail/Chip-Resistor-Surface-Mount_Viking-Tech-ARG03FTC0100_C217691.html" H 8400 3100 50  0001 C CNN "Link"
+F 6 "ARG03FTC0100" H 8400 3100 50  0001 C CNN "MPN"
 	1    8400 3100
 	0    -1   -1   0
