File: osab.sch (KiCad schematic (older format))
At the start: 88 parts, among them CON1 TF-01A, CON2 PJ-3420-A-SMT, CON3 TYPE-C-31-M-12, Q1 BC847B, SW1 PPP, SW10 RESET, SW2 VOL-, SW3 VOL+, SW4 CHAP-, SW5 CHAP+, SW6 OT/NT, SW7 BOOK-, SW8 BOOK+, SW9 BUTTON_LOCK, U1 VS1000, U2 ME6211C33M5G-N, U3 25LC640A, U4 TP4055, U5 MF5853CS, U6 TCS7191, Y1 12MHz

Commit message: production: Changed all 20R resistors to 0603
Parts:
- R24, R25: Link https://lcsc.com/product-detail/Others_Viking-Tech-ARG05FTC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 -> https://lcsc.com/product-detail/Chip-Resistor-Surface-Mount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; MPN ARG05FTC0200 -> ARG03FTC0200
Changed lines of the file:
@@
 F 1 "20" V 7650 3650 50  0000 C CNN
 F 2 "Resistor_SMD:R_0603_1608Metric" V 7580 3650 50  0001 C CNN
-F 3 "https://datasheet.lcsc.com/szlcsc/1810261818_Viking-Tech-ARG05FTC0200_C218421.pdf" H 7650 3650 50  0001 C CNN
+F 3 "https://datasheet.lcsc.com/lcsc/1811091511_Viking-Tech-ARG03FTC0200_C217873.pdf" H 7650 3650 50  0001 C CNN
 F 4 "Included in KiCad" H 7650 3650 50  0001 C CNN "3D-model"
-F 5 "https://lcsc.com/product-detail/Others_Viking-Tech-ARG05FTC0200_C218421.html" H 7650 3650 50  0001 C CNN "Link"
-F 6 "ARG05FTC0200" H 7650 3650 50  0001 C CNN "MPN"
+F 5 "https://lcsc.com/product-detail/Chip-Resistor-Surface-Mount_Viking-Tech-ARG03FTC0200_C217873.html" H 7650 3650 50  0001 C CNN "Link"
+F 6 "ARG03FTC0200" H 7650 3650 50  0001 C CNN "MPN"
 	1    7650 3650
 	-1   0    0    1
@@
 F 1 "20" V 7850 3650 50  0000 C CNN
 F 2 "Resistor_SMD:R_0603_1608Metric" V 7780 3650 50  0001 C CNN
-F 3 "https://datasheet.lcsc.com/szlcsc/1810261818_Viking-Tech-ARG05FTC0200_C218421.pdf" H 7850 3650 50  0001 C CNN
+F 3 "https://datasheet.lcsc.com/lcsc/1811091511_Viking-Tech-ARG03FTC0200_C217873.pdf" H 7850 3650 50  0001 C CNN
 F 4 "Included in KiCad" H 7850 3650 50  0001 C CNN "3D-model"
-F 5 "https://lcsc.com/product-detail/Others_Viking-Tech-ARG05FTC0200_C218421.html" H 7850 3650 50  0001 C CNN "Link"
-F 6 "ARG05FTC0200" H 7850 3650 50  0001 C CNN "MPN"
+F 5 "https://lcsc.com/product-detail/Chip-Resistor-Surface-Mount_Viking-Tech-ARG03FTC0200_C217873.html" H 7850 3650 50  0001 C CNN "Link"
+F 6 "ARG03FTC0200" H 7850 3650 50  0001 C CNN "MPN"
 	1    7850 3650
 	-1   0    0    1

Commit message: production: Changed all 470R resistors to 0603
Parts:
- R28, R29: Link https://lcsc.com/product-detail/Others_Viking-Tech-ARG05FTC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 -> https://lcsc.com/product-detail/Chip-Resistor-Surface-Mount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; MPN ARG05FTC4700 -> ARG03FTC4700
Changed lines of the file:
@@
 F 1 "470" V 8450 3300 50  0000 C CNN
 F 2 "Resistor_SMD:R_0603_1608Metric" V 8380 3300 50  0001 C CNN
-F 3 "https://datasheet.lcsc.com/szlcsc/1810261818_Viking-Tech-ARG05FTC4700_C218590.pdf" H 8450 3300 50  0001 C CNN
+F 3 "https://datasheet.lcsc.com/lcsc/1811091511_Viking-Tech-ARG03FTC4700_C218042.pdf" H 8450 3300 50  0001 C CNN
 F 4 "Included in KiCad" H 8450 3300 50  0001 C CNN "3D-model"
-F 5 "https://lcsc.com/product-detail/Others_Viking-Tech-ARG05FTC4700_C218590.html" H 8450 3300 50  0001 C CNN "Link"
-F 6 "ARG05FTC4700" H 8450 3300 50  0001 C CNN "MPN"
+F 5 "https://lcsc.com/product-detail/Chip-Resistor-Surface-Mount_Viking-Tech-ARG03FTC4700_C218042.html" H 8450 3300 50  0001 C CNN "Link"
+F 6 "ARG03FTC4700" H 8450 3300 50  0001 C CNN "MPN"
 	1    8450 3300
 	0    -1   -1   0
@@
 F 1 "470" V 8450 3450 50  0000 C CNN
 F 2 "Resistor_SMD:R_0603_1608Metric" V 8380 3450 50  0001 C CNN
-F 3 "https://datasheet.lcsc.com/szlcsc/1810261818_Viking-Tech-ARG05FTC4700_C218590.pdf" H 8450 3450 50  0001 C CNN
+F 3 "https://datasheet.lcsc.com/lcsc/1811091511_Viking-Tech-ARG03FTC4700_C218042.pdf" H 8450 3450 50  0001 C CNN
 F 4 "Included in KiCad" H 8450 3450 50  0001 C CNN "3D-model"
-F 5 "https://lcsc.com/product-detail/Others_Viking-Tech-ARG05FTC4700_C218590.html" H 8450 3450 50  0001 C CNN "Link"
-F 6 "ARG05FTC4700" H 8450 3450 50  0001 C CNN "MPN"
+F 5 "https://lcsc.com/product-detail/Chip-Resistor-Surface-Mount_Viking-Tech-ARG03FTC4700_C218042.html" H 8450 3450 50  0001 C CNN "Link"
+F 6 "ARG03FTC4700" H 8450 3450 50  0001 C CNN "MPN"
 	1    8450 3450
 	0    -1   -1   0

Commit message: production: Changed 5k1 resistor to 0603
Parts:
- R21: Link https://lcsc.com/product-detail/Others_Viking-Tech-ARG05FTC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 -> https://lcsc.com/product-detail/Chip-Resistor-Surface-Mount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; MPN ARG05FTC5101 -> ARG03FTC5101
Changed lines of the file:
@@
 F 1 "5k1 1%" V 9950 5200 50  0000 C CNN
 F 2 "Resistor_SMD:R_0603_1608Metric" V 9880 5100 50  0001 C CNN
-F 3 "https://datasheet.lcsc.com/szlcsc/1810261825_Viking-Tech-ARG05FTC5101_C218638.pdf" H 9950 5100 50  0001 C CNN
+F 3 "https://datasheet.lcsc.com/lcsc/1811091612_Viking-Tech-ARG03FTC5101_C218090.pdf" H 9950 5100 50  0001 C CNN
 F 4 "Included in KiCad" H 9950 5100 50  0001 C CNN "3D-model"
-F 5 "https://lcsc.com/product-detail/Others_Viking-Tech-ARG05FTC5101_C218638.html" H 9950 5100 50  0001 C CNN "Link"
-F 6 "ARG05FTC5101" H 9950 5100 50  0001 C CNN "MPN"
+F 5 "https://lcsc.com/product-detail/Chip-Resistor-Surface-Mount_Viking-Tech-ARG03FTC5101_C218090.html" H 9950 5100 50  0001 C CNN "Link"
+F 6 "ARG03FTC5101" H 9950 5100 50  0001 C CNN "MPN"
 	1    9950 5100
 	1    0    0    -1

Commit message: production: Changed all 100R resistors to 0603
Parts:
- R36, R37: Link https://lcsc.com/product-detail/Others_Viking-Tech-ARG05FTC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 -> https://lcsc.com/product-detail/Chip-Resistor-Surface-Mount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; MPN ARG05FTC1000 -> ARG03FTC1000
Changed lines of the file:
@@
 F 1 "100" V 7450 4500 50  0000 C CNN
 F 2 "Resistor_SMD:R_0603_1608Metric" V 7380 4500 50  0001 C CNN
-F 3 "https://datasheet.lcsc.com/szlcsc/1810261818_Viking-Tech-ARG05FTC1000_C217766.pdf" H 7450 4500 50  0001 C CNN
+F 3 "https://datasheet.lcsc.com/lcsc/1811091620_Viking-Tech-ARG03FTC1000_C217683.pdf" H 7450 4500 50  0001 C CNN
 F 4 "Included in KiCad" H 7450 4500 50  0001 C CNN "3D-model"
-F 5 "https://lcsc.com/product-detail/Others_Viking-Tech-ARG05FTC1000_C217766.html" H 7450 4500 50  0001 C CNN "Link"
-F 6 "ARG05FTC1000" H 7450 4500 50  0001 C CNN "MPN"
+F 5 "https://lcsc.com/product-detail/Chip-Resistor-Surface-Mount_Viking-Tech-ARG03FTC1000_C217683.html" H 7450 4500 50  0001 C CNN "Link"
+F 6 "ARG03FTC1000" H 7450 4500 50  0001 C CNN "MPN"
 	1    7450 4500
 	0    1    1    0
@@
 F 1 "100" V 7200 4400 50  0000 C CNN
 F 2 "Resistor_SMD:R_0603_1608Metric" V 7130 4400 50  0001 C CNN
-F 3 "https://datasheet.lcsc.com/szlcsc/1810261818_Viking-Tech-ARG05FTC1000_C217766.pdf" H 7200 4400 50  0001 C CNN
+F 3 "https://datasheet.lcsc.com/lcsc/1811091620_Viking-Tech-ARG03FTC1000_C217683.pdf" H 7200 4400 50  0001 C CNN
 F 4 "Included in KiCad" H 7200 4400 50  0001 C CNN "3D-model"
-F 5 "https://lcsc.com/product-detail/Others_Viking-Tech-ARG05FTC1000_C217766.html" H 7200 4400 50  0001 C CNN "Link"
-F 6 "ARG05FTC1000" H 7200 4400 50  0001 C CNN "MPN"
+F 5 "https://lcsc.com/product-detail/Chip-Resistor-Surface-Mount_Viking-Tech-ARG03FTC1000_C217683.html" H 7200 4400 50  0001 C CNN "Link"
+F 6 "ARG03FTC1000" H 7200 4400 50  0001 C CNN "MPN"
 	1    7200 4400
 	0    1    1    0

Commit message: production: Changed 33k resistor to 0603
Parts:
- R33: Link https://lcsc.com/product-detail/Others_Viking-Tech-ARG05FTC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 -> https://lcsc.com/product-detail/Chip-Resistor-Surface-Mount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; MPN ARG05FTC3302 -> ARG03FTC3302
Changed lines of the file:
@@
 F 1 "33k" V 11000 4050 50  0000 C CNN
 F 2 "Resistor_SMD:R_0603_1608Metric" V 10930 4050 50  0001 C CNN
-F 3 "https://datasheet.lcsc.com/szlcsc/1810261826_Viking-Tech-ARG05FTC3302_C218519.pdf" H 11000 4050 50  0001 C CNN
+F 3 "https://datasheet.lcsc.com/lcsc/1811091520_Viking-Tech-ARG03FTC3302_C217971.pdf" H 11000 4050 50  0001 C CNN
 F 4 "Included in KiCad" H 11000 4050 50  0001 C CNN "3D-model"
-F 5 "https://lcsc.com/product-detail/Others_Viking-Tech-ARG05FTC3302_C218519.html" H 11000 4050 50  0001 C CNN "Link"
-F 6 "ARG05FTC3302" H 11000 4050 50  0001 C CNN "MPN"
+F 5 "https://lcsc.com/product-detail/Chip-Resistor-Surface-Mount_Viking-Tech-ARG03FTC3302_C217971.html" H 11000 4050 50  0001 C CNN "Link"
+F 6 "ARG03FTC3302" H 11000 4050 50  0001 C CNN "MPN"
 	1    11000 4050
 	1    0    0    -1

Commit message: production: Changed 25LC640A to CAT25640
Parts:
- U3: value 25LC640A -> CAT25640; symbol osab:25LC640A -> osab:CAT25640; Link https://lcsc.com/product-detail/EEPROM_Microchip-Tech-25LC6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 -> https://lcsc.com/product-detail/EEPROM_onsemi-CAT25640VI-GT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; MPN 25LC640T-I/SN -> CAT25640VI-GT3
Changed lines of the file:
@@
 $EndComp
 $Comp
-L osab:25LC640A U3
+L osab:CAT25640 U3
 U 1 1 54C921E7
 P 6100 3700
 F 0 "U3" H 5900 3700 60  0000 C CNN
-F 1 "25LC640A" H 6100 3200 60  0000 C CNN
+F 1 "CAT25640" H 6100 3200 60  0000 C CNN
 F 2 "Package_SO:SOIC-8_3.9x4.9mm_P1.27mm" H 6100 3700 60  0001 C CNN
-F 3 "https://datasheet.lcsc.com/szlcsc/1809192127_Microchip-Tech-25LC640T-I-SN_C5464.pdf" H 6100 3700 60  0001 C CNN
+F 3 "https://datasheet.lcsc.com/lcsc/1809171606_onsemi-CAT25640VI-GT3_C153776.pdf" H 6100 3700 60  0001 C CNN
 F 4 "Included in KiCad" H 6100 3700 50  0001 C CNN "3D-model"
-F 5 "https://lcsc.com/product-detail/EEPROM_Microchip-Tech-25LC640T-I-SN_C5464.html" H 6100 3700 50  0001 C CNN "Link"
-F 6 "25LC640T-I/SN" H 6100 3700 50  0001 C CNN "MPN"
+F 5 "https://lcsc.com/product-detail/EEPROM_onsemi-CAT25640VI-GT3_C153776.html" H 6100 3700 50  0001 C CNN "Link"
+F 6 "CAT25640VI-GT3" H 6100 3700 50  0001 C CNN "MPN"
 	1    6100 3700
 	1    0    0    -1

Commit message: production: Replaced TCS7191 with PAM8302A
Parts:
- U6: value TCS7191 -> PAM8302A; symbol osab:TCS7191 -> osab:PAM8302A; Link https://www.digchip.com/datasheets/quote.php?action=search&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 -> https://lcsc.com/product-detail/Audio-Power-OpAmps_Diodes-I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; MPN TCS7191B -> PAM8302AASCR
Changed lines of the file:
@@
 U 1 1 54D41AFF
 P 6750 3900
-F 0 "BOOT1" V 6750 4100 50  0000 C CNN
+F 0 "BOOT1 - REMOVE" V 6750 4100 50  0000 C CNN
 F 1 "BOOT" H 6750 3820 50  0001 C CNN
 F 2 "OSAB:Terminals_2_SMD" H 6750 3900 60  0001 C CNN
@@
 $EndComp
 $Comp
-L osab:TCS7191 U6
+L osab:PAM8302A U6
 U 1 1 54D59A57
 P 9750 3000
 F 0 "U6" H 9900 3200 60  0000 C CNN
-F 1 "TCS7191" H 9750 2450 60  0000 C CNN
+F 1 "PAM8302A" H 9750 2450 60  0000 C CNN
 F 2 "Package_SO:MSOP-8_3x3mm_P0.65mm" H 9800 3200 60  0001 C CNN
-F 3 "https://datasheetspdf.com/pdf-file/869014/TCS/TCS7191B/1" H 9800 3200 60  0001 C CNN
+F 3 "https://datasheet.lcsc.com/lcsc/1809192050_Diodes-Incorporated-PAM8302AASCR_C113367.pdf" H 9800 3200 60  0001 C CNN
 F 4 "Included in KiCad" H 9750 3000 50  0001 C CNN "3D-model"
-F 5 "https://www.digchip.com/datasheets/quote.php?action=search&pn=TCS7191B" H 9750 3000 50  0001 C CNN "Link"
-F 6 "TCS7191B" H 9750 3000 50  0001 C CNN "MPN"
+F 5 "https://lcsc.com/product-detail/Audio-Power-OpAmps_Diodes-Incorporated-PAM8302AASCR_C113367.html" H 9750 3000 50  0001 C CNN "Link"
+F 6 "PAM8302AASCR" H 9750 3000 50  0001 C CNN "MPN"
 	1    9750 3000
 	1    0    0    -1

Commit message: production: New LEDs
Parts:
- D1: footprint LED_SMD:LED_0805_2012Metric -> Custom 1.6x0.6x1.1mm footprint; Link https://lcsc.com/product-detail/Light-Emitting-Diodes-LED_Everlight-Elec-17-21-BHC-XL2M2TY-3T_C72035.html -> https://lcsc.com/product-detail/Light-Emitting-Diodes-LED_EKINGLUX-E6X0602CWAY1UDA_C375469.html; MPN 17-21/BHC-XL2M2TY/3T -> E6X0602CWAY1UDA
- D2: footprint LED_SMD:LED_0805_2012Metric -> Custom 0602 footprint; Link https://lcsc.com/product-detail/Light-Emitting-Diodes-LED_0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 -> https://lcsc.com/product-detail/Light-Emitting-Diodes-LED_L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; MPN 17-21SURC/S530-A3/TR8 -> LTST-S270KRKT
Changed lines of the file:
@@
 F 0 "D2" V 8200 4500 50  0000 L CNN
 F 1 "Charge LED" V 8300 4100 50  0000 L CNN
-F 2 "LED_SMD:LED_0805_2012Metric" V 8300 4600 50  0001 C CNN
-F 3 "https://datasheet.lcsc.com/szlcsc/1811061932_Everlight-Elec-17-21SURC-S530-A3-TR8_C72037.pdf" V 8300 4600 50  0001 C CNN
-F 4 "https://lcsc.com/product-detail/Light-Emitting-Diodes-LED_0805-Red-LED-Iv-61mcd-Typ-atIF-20mA_C72037.html" H 8300 4600 50  0001 C CNN "Link"
-F 5 "17-21SURC/S530-A3/TR8" H 8300 4600 50  0001 C CNN "MPN"
+F 2 "Custom 0602 footprint" V 8300 4600 50  0001 C CNN
+F 3 "https://datasheet.lcsc.com/lcsc/1810231514_Lite-On-LTST-S270KRKT_C125114.pdf" V 8300 4600 50  0001 C CNN
+F 4 "https://lcsc.com/product-detail/Light-Emitting-Diodes-LED_Lite-On-LTST-S270KRKT_C125114.html" H 8300 4600 50  0001 C CNN "Link"
+F 5 "LTST-S270KRKT" H 8300 4600 50  0001 C CNN "MPN"
 F 6 "Included in KiCad" H 8300 4600 50  0001 C CNN "3D-model"
 	1    8300 4600
@@
 F 0 "D1" H 2100 4250 50  0000 L CNN
 F 1 "Status LED" H 2100 4150 50  0000 L CNN
-F 2 "LED_SMD:LED_0805_2012Metric" V 2250 4200 50  0001 C CNN
-F 3 "https://datasheet.lcsc.com/szlcsc/1809192317_Everlight-Elec-17-21-BHC-XL2M2TY-3T_C72035.pdf" V 2250 4200 50  0001 C CNN
-F 4 "https://lcsc.com/product-detail/Light-Emitting-Diodes-LED_Everlight-Elec-17-21-BHC-XL2M2TY-3T_C72035.html" H 2250 4200 50  0001 C CNN "Link"
-F 5 "17-21/BHC-XL2M2TY/3T" H 2250 4200 50  0001 C CNN "MPN"
+F 2 "Custom 1.6x0.6x1.1mm footprint" V 2250 4200 50  0001 C CNN
+F 3 "https://datasheet.lcsc.com/lcsc/2105241210_EKINGLUX-E6X0602CWAY1UDA_C375469.pdf" V 2250 4200 50  0001 C CNN
+F 4 "https://lcsc.com/product-detail/Light-Emitting-Diodes-LED_EKINGLUX-E6X0602CWAY1UDA_C375469.html" H 2250 4200 50  0001 C CNN "Link"
+F 5 "E6X0602CWAY1UDA" H 2250 4200 50  0001 C CNN "MPN"
 F 6 "Included in KiCad" H 2250 4200 50  0001 C CNN "3D-model"
 	1    2250 4200
