File: osab.kicad_pcb (KiCad board)
At the start: 2 copper layers, 50 x 75 mm, 98 parts, among them CON1 TF-01A, CON2 PJ-3420-A-SMT, CON3 TYPE-C-31-M-12, Q1 BC847B, Q2 BC847B, SW1 PPP, SW10 RESET, SW11 Torch, SW2 VOL-, SW3 VOL+, SW4 CHAP-, SW5 CHAP+, SW6 OT/NT, SW7 BOOK-, SW8 BOOK+, SW9 XKB5858-Z-F, U1 VS1000, U2 ME6211C33M5G-N, U3 CAT25640, U4 TP4055, U5 MF5853CS, U6 PAM8302AAS, Y1 12MHz

Commit message: production: Routing tracks...
Routing:
- net Net-(R16-Pad2): track 11.7 -> 37.6 mm, vias 0 -> 2
- net VDD: track 94.7 -> 99.7 mm, vias 1 -> 2
- net Net-(R2-Pad1): track 56.0 -> 54.9 mm

Commit message: production: Routing tracks...
Routing:
- net Net-(R33-Pad2): track 0.00 -> 48.2 mm, vias 0 -> 6
- net VDD: track 99.7 -> 102.7 mm

Commit message: production: Routing tracks...
Routing:
- net AVDD: track 24.6 -> 33.9 mm
Changed lines of the file:
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@@
   (segment (start 143.175 80.55) (end 143.425 80.8) (width 0.3) (layer "F.Cu") (net 9))
   (segment (start 141.27952 88.17452) (end 143.577663 88.17452) (width 0.16) (layer "F.Cu") (net 10))
+  (segment (start 139.16 81.25) (end 138.89 81.52) (width 0.3) (layer "F.Cu") (net 10))
+  (segment (start 138.9 82.55) (end 139.2 82.25) (width 0.3) (layer "F.Cu") (net 10))
   (segment (start 141.75 82.25) (end 141.9 82.1) (width 0.3) (layer "F.Cu") (net 10))
   (segment (start 144.67952 90.57048) (end 143.925 91.325) (width 0.16) (layer "F.Cu") (net 10))
+  (segment (start 138.89548 86.07548) (end 139.12548 86.07548) (width 0.3) (layer "F.Cu") (net 10))
   (segment (start 137.75 87.1625) (end 137.75 86.324639) (width 0.3) (layer "F.Cu") (net 10))
   (segment (start 141.43516 84.75) (end 141.444182 84.759022) (width 0.3) (layer "F.Cu") (net 10))
@@
   (segment (start 143.425 79.312507) (end 143.425 79.1) (width 0.3) (layer "F.Cu") (net 10))
   (segment (start 141.487507 81.25) (end 143.425 79.312507) (width 0.3) (layer "F.Cu") (net 10))
+  (segment (start 138.89 81.52) (end 138.89 81.94) (width 0.3) (layer "F.Cu") (net 10))
+  (segment (start 139.32 84.75) (end 138.9 84.33) (width 0.3) (layer "F.Cu") (net 10))
+  (segment (start 140.1625 84.75) (end 139.32 84.75) (width 0.3) (layer "F.Cu") (net 10))
+  (segment (start 140.1625 81.25) (end 139.16 81.25) (width 0.3) (layer "F.Cu") (net 10))
   (segment (start 143.362507 79.3) (end 143.45 79.3) (width 0.3) (layer "F.Cu") (net 10))
+  (segment (start 138.89548 84.89452) (end 139.04 84.75) (width 0.3) (layer "F.Cu") (net 10))
   (segment (start 140.1625 84.75) (end 141.43516 84.75) (width 0.3) (layer "F.Cu") (net 10))
   (segment (start 140.1625 81.25) (end 141.487507 81.25) (width 0.3) (layer "F.Cu") (net 10))
+  (segment (start 139.04 84.75) (end 140.1625 84.75) (width 0.3) (layer "F.Cu") (net 10))
   (segment (start 140.47 87.42) (end 140.525 87.42) (width 0.3) (layer "F.Cu") (net 10))
+  (segment (start 137.999159 86.07548) (end 138.89548 86.07548) (width 0.3) (layer "F.Cu") (net 10))
+  (segment (start 138.9 84.33) (end 138.9 82.55) (width 0.3) (layer "F.Cu") (net 10))
   (segment (start 141.9 82.1) (end 143.425 82.1) (width 0.3) (layer "F.Cu") (net 10))
-  (segment (start 137.999159 86.07548) (end 139.12548 86.07548) (width 0.3) (layer "F.Cu") (net 10))
   (segment (start 142.425 91.325) (end 144.2 91.325) (width 0.16) (layer "F.Cu") (net 10))
   (segment (start 141.444182 84.759022) (end 141.584022 84.759022) (width 0.3) (layer "F.Cu") (net 10))
+  (segment (start 138.89 81.94) (end 139.2 82.25) (width 0.3) (layer "F.Cu") (net 10))
   (segment (start 139.12548 86.07548) (end 140.47 87.42) (width 0.3) (layer "F.Cu") (net 10))
   (segment (start 140.1625 82.25) (end 141.75 82.25) (width 0.3) (layer "F.Cu") (net 10))
@@
   (segment (start 141.584022 84.759022) (end 142.725 85.9) (width 0.3) (layer "F.Cu") (net 10))
   (segment (start 140.525 87.42) (end 141.27952 88.17452) (width 0.16) (layer "F.Cu") (net 10))
+  (segment (start 138.89548 86.07548) (end 138.89548 84.89452) (width 0.3) (layer "F.Cu") (net 10))
+  (segment (start 139.2 82.25) (end 140.1625 82.25) (width 0.3) (layer "F.Cu") (net 10))
   (segment (start 143.425 82.087493) (end 143.425 82.4) (width 0.3) (layer "F.Cu") (net 10))
   (segment (start 152.19 115.69) (end 155.03 115.69) (width 0.25) (layer "F.Cu") (net 11))

Commit message: production: Routing tracks...
Parts:
- moved R38 0.20 mm to (145.3, 72.5)
- moved Q2 0.10 mm to (142.8, 64.8)
Routing:
- net Net-(R38-Pad1): track 21.3 -> 49.7 mm
- net Net-(R37-Pad2): track 41.9 -> 59.9 mm, vias 6 -> 2

Commit message: production: Routing tracks...
Parts:
- moved R16 7.97 mm to (131.9, 74.2), turned to 180 degrees
- moved C8 0.73 mm to (135.8, 76.3), turned to 90 degrees
- moved R38 0.50 mm to (144.8, 72.5)
Routing:
- net Net-(R6-Pad1): track 8.20 -> 50.0 mm, vias 0 -> 2
- net Net-(R8-Pad1): track 2.17 -> 31.6 mm, vias 0 -> 2
- net Net-(R16-Pad2): track 37.6 -> 62.5 mm, vias 2 -> 4
- net Net-(R2-Pad1): track 54.9 -> 65.3 mm
- net VDD: track 102.7 -> 107.2 mm
- net Net-(CON3-PadA6): track 3.24 -> 5.93 mm
- net Net-(R1-Pad2): track 16.7 -> 15.4 mm
- net GND: track 110.6 -> 109.4 mm, vias 43 -> 44
- net Net-(R33-Pad2): track 48.2 -> 49.0 mm

Commit message: production: Routing tracks...
Routing:
- net Net-(R5-Pad1): track 6.70 -> 82.1 mm, vias 0 -> 6
- net Net-(R33-Pad2): track 49.0 -> 50.4 mm

Commit message: production: Routing tracks...
Routing:
- net Net-(R7-Pad1): track 2.17 -> 94.8 mm, vias 0 -> 4
- net Net-(R16-Pad2): track 62.5 -> 61.2 mm
- net GND: track 109.4 -> 110.2 mm, vias 44 -> 45

Commit message: production: Routing tracks...
Routing:
- net Net-(R4-Pad1): track 0.00 -> 45.6 mm, vias 0 -> 2
- net Net-(R6-Pad1): track 50.1 -> 51.9 mm
- net VDD: track 107.2 -> 108.5 mm
- net Net-(R8-Pad1): track 31.6 -> 32.5 mm
