File: osab.kicad_sch (KiCad schematic)
At the start: 98 parts, among them CON1 TF-01A, CON2 PJ-3420-A-SMT, CON3 TYPE-C-31-M-12, Q1 BC847B, Q2 BC847B, SW1 PPP, SW10 RESET, SW11 Torch, SW2 VOL-, SW3 VOL+, SW4 CHAP-, SW5 CHAP+, SW6 OT/NT, SW7 BOOK-, SW8 BOOK+, SW9 XKB5858-Z-F, U1 VS1000, U2 ME6211C33M5G-N, U3 CAT25640, U4 TP4055, U5 MF5853CS, U6 PAM8302AAS, Y1 12MHz

Commit message: production: New status LED and speaker connector
Parts:
- D1: footprint OSAB:0602-LED -> OSAB:0805-LED; LCSC C375469 -> C693902; Link https://lcsc.com/product-detail/Light-Emitting-Diodes-LED_E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 -> https://lcsc.com/product-detail/Light-Emitting-Diodes-LED_M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; MPN E6X0602CWAY1UDA -> MHS171WDT-C2
- SPEAKER1: footprint OSAB:HYCW02-WF02-125B -> OSAB:WAFER-125W-2P; LCSC C2939022 -> C2840410; Link https://lcsc.com/product-detail/Wire-To-Board-Wire-To-Wire-Connector_HOAUC-HYCW02-WF02-125B_C2939022.html -> https://lcsc.com/product-detail/Wire-To-Board-Wire-To-Wire-Connector_XUNPU-WAFER-125W-2P_C2840410.html; MPN HYCW02-WF02-125B -> WAFER-125W-2P
Changed lines of the file:
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@@
       (effects (font (size 1.27 1.27)) (justify left) hide)
     )
-    (property "Footprint" "OSAB:HYCW02-WF02-125B" (id 2) (at 276.86 78.74 0)
-      (effects (font (size 1.27 1.27)) hide)
-    )
-    (property "Datasheet" "https://datasheet.lcsc.com/lcsc/2201261500_HOAUC-HYCW02-WF02-125B_C2939022.pdf" (id 3) (at 276.86 78.74 0)
-      (effects (font (size 1.27 1.27)) hide)
-    )
-    (property "Link" "https://lcsc.com/product-detail/Wire-To-Board-Wire-To-Wire-Connector_HOAUC-HYCW02-WF02-125B_C2939022.html" (id 5) (at 276.86 78.74 0)
-      (effects (font (size 1.27 1.27)) hide)
-    )
-    (property "MPN" "HYCW02-WF02-125B" (id 6) (at 276.86 78.74 0)
-      (effects (font (size 1.27 1.27)) hide)
-    )
-    (property "LCSC" "C2939022" (id 7) (at 276.86 78.74 0)
+    (property "Footprint" "OSAB:WAFER-125W-2P" (id 2) (at 276.86 78.74 0)
+      (effects (font (size 1.27 1.27)) hide)
+    )
+    (property "Datasheet" "https://datasheet.lcsc.com/lcsc/2202132000_XUNPU-WAFER-125W-2P_C2840410.pdf" (id 3) (at 276.86 78.74 0)
+      (effects (font (size 1.27 1.27)) hide)
+    )
+    (property "Link" "https://lcsc.com/product-detail/Wire-To-Board-Wire-To-Wire-Connector_XUNPU-WAFER-125W-2P_C2840410.html" (id 5) (at 276.86 78.74 0)
+      (effects (font (size 1.27 1.27)) hide)
+    )
+    (property "MPN" "WAFER-125W-2P" (id 6) (at 276.86 78.74 0)
+      (effects (font (size 1.27 1.27)) hide)
+    )
+    (property "LCSC" "C2840410" (id 7) (at 276.86 78.74 0)
       (effects (font (size 1.524 1.524)) hide)
     )
@@
     (property "Reference" "D1" (id 0) (at 118.11 166.37 90))
     (property "Value" "Status LED" (id 1) (at 114.3 163.83 90))
-    (property "Footprint" "OSAB:0602-LED" (id 2) (at 120.65 166.37 0)
-      (effects (font (size 1.27 1.27)) hide)
-    )
-    (property "Datasheet" "https://datasheet.lcsc.com/lcsc/2105241210_EKINGLUX-E6X0602CWAY1UDA_C375469.pdf" (id 3) (at 120.65 166.37 0)
-      (effects (font (size 1.27 1.27)) hide)
-    )
-    (property "Link" "https://lcsc.com/product-detail/Light-Emitting-Diodes-LED_EKINGLUX-E6X0602CWAY1UDA_C375469.html" (id 4) (at 120.65 166.37 0)
-      (effects (font (size 1.27 1.27)) hide)
-    )
-    (property "MPN" "E6X0602CWAY1UDA" (id 5) (at 120.65 166.37 0)
-      (effects (font (size 1.27 1.27)) hide)
-    )
-    (property "LCSC" "C375469" (id 7) (at 120.65 166.37 90)
+    (property "Footprint" "OSAB:0805-LED" (id 2) (at 120.65 166.37 0)
+      (effects (font (size 1.27 1.27)) hide)
+    )
+    (property "Datasheet" "https://datasheet.lcsc.com/lcsc/2007030604_MEIHUA-MHS171WDT-C2_C693902.pdf" (id 3) (at 120.65 166.37 0)
+      (effects (font (size 1.27 1.27)) hide)
+    )
+    (property "Link" "https://lcsc.com/product-detail/Light-Emitting-Diodes-LED_MEIHUA-MHS171WDT-C2_C693902.html" (id 4) (at 120.65 166.37 0)
+      (effects (font (size 1.27 1.27)) hide)
+    )
+    (property "MPN" "MHS171WDT-C2" (id 5) (at 120.65 166.37 0)
+      (effects (font (size 1.27 1.27)) hide)
+    )
+    (property "LCSC" "C693902" (id 7) (at 120.65 166.37 90)
       (effects (font (size 1.524 1.524)) hide)
     )
@@
     )
     (path "/0d36bc22-9af2-4964-ab81-0226abd299f7"
-      (reference "D1") (unit 1) (value "Status LED") (footprint "OSAB:0602-LED")
+      (reference "D1") (unit 1) (value "Status LED") (footprint "OSAB:0805-LED")
     )
     (path "/3a20fa27-1c24-4388-b4e8-5dff7e0ea510"
@@
     )
     (path "/00000000-0000-0000-0000-00005e03f86a"
-      (reference "SPEAKER1") (unit 1) (value "Conn_01x02") (footprint "OSAB:HYCW02-WF02-125B")
+      (reference "SPEAKER1") (unit 1) (value "Conn_01x02") (footprint "OSAB:WAFER-125W-2P")
     )
     (path "/00000000-0000-0000-0000-0000543f883c"
